File: Hardware/Cantaloupe.sch (KiCad schematic (older format))
At the start: 146 parts, among them J1 USB_C_Receptacle_PD, J2 Bat, J3 OLED, J4 USB_C_Receptacle_PD, J5 Bat, J6 OLED, SW1 MX, SW10 MX, SW11 MX, SW12 MX, SW13 MX, SW14 MX, SW15 MX, SW16 MX, SW17 MX, SW18 MX, SW19 MX, SW2 MX, SW20 MX, SW21 MX, SW22 MX, SW23 MX, SW24 MX, SW25 MX, SW26 MX, SW27 MX, SW28 MX, SW29 MX, SW3 MX, SW30 MX, SW31 5_Way_Tactile_Switch, SW32 Rotary_Encoder_Switch, SW33 5_Way_Tactile_Switch_R, SW34 Reset, SW35 MX, SW36 MX, SW37 MX, SW38 MX, SW39 MX, SW4 MX, SW40 MX, SW41 MX, SW42 MX, SW43 MX, SW44 MX, SW45 MX, SW46 MX, SW47 MX, SW48 MX, SW49 MX, SW5 MX, SW50 MX, SW51 MX, SW52 MX, SW53 MX, SW54 MX, SW55 MX, SW56 MX, SW57 MX, SW58 MX, SW59 MX, SW6 MX, SW60 MX, SW61 MX, SW62 MX, SW63 MX, SW65 MX, SW66 Rotary_Encoder_Switch, SW67 Reset, SW7 MX, SW8 MX, SW9 MX, U1 ProMicro, U2 ProMicro

Commit message: Added BOM
Parts:
- R1: value 4.7k -> 10k
- R2: renamed from R4; value 4.7k -> 10k
- renumbered SW32 to SW31, SW31 to SW32, SW34 to SW33, SW35 to SW34, SW36 to SW35, SW37 to SW36, SW38 to SW37, SW39 to SW38, SW40 to SW39, SW41 to SW40, SW42 to SW41, SW43 to SW42, SW44 to SW43, SW45 to SW44, SW46 to SW45, SW47 to SW46, SW48 to SW47, SW49 to SW48, SW50 to SW49, SW51 to SW50, SW52 to SW51, SW53 to SW52, SW58 to SW53, SW63 to SW58, SW65 to SW63, SW66 to SW64, SW33 to SW65, SW67 to SW66
Changed lines of the file:
@@
 Connection ~ 3200 3200
 $Comp
-L Switch:SW_Push SW67
+L Switch:SW_Push SW66
 U 1 1 609DB9B8
 P 8150 5800
-F 0 "SW67" H 8150 6085 50  0000 C CNN
+F 0 "SW66" H 8150 6085 50  0000 C CNN
 F 1 "Reset" H 8150 5994 50  0000 C CNN
 F 2 "Button_Switch_SMD:SW_SPST_TL3342" H 8150 6000 50  0001 C CNN
@@
 $EndComp
 $Comp
-L Device:R_Small R4
+L Device:R_Small R2
 U 1 1 609DB9BE
 P 7950 5700
-F 0 "R4" H 7800 5750 50  0000 L CNN
-F 1 "4.7k" H 7750 5650 50  0000 L CNN
+F 0 "R2" H 7800 5750 50  0000 L CNN
+F 1 "10k" H 7750 5650 50  0000 L CNN
 F 2 "Resistor_SMD:R_0603_1608Metric_Pad1.05x0.95mm_HandSolder" H 7950 5700 50  0001 C CNN
 F 3 "~" H 7950 5700 50  0001 C CNN
@@
 $EndComp
 $Comp
-L Switch:SW_Push SW34
+L Switch:SW_Push SW33
 U 1 1 5E7DD54D
 P 8050 2950
-F 0 "SW34" H 8050 3235 50  0000 C CNN
+F 0 "SW33" H 8050 3235 50  0000 C CNN
 F 1 "Reset" H 8050 3144 50  0000 C CNN
 F 2 "Button_Switch_SMD:SW_SPST_TL3342" H 8050 3150 50  0001 C CNN
@@
 P 7850 2850
 F 0 "R1" H 7700 2900 50  0000 L CNN
-F 1 "4.7k" H 7650 2800 50  0000 L CNN
+F 1 "10k" H 7650 2800 50  0000 L CNN
 F 2 "Resistor_SMD:R_0603_1608Metric_Pad1.05x0.95mm_HandSolder" H 7850 2850 50  0001 C CNN
 F 3 "~" H 7850 2850 50  0001 C CNN
@@
 COL7
 $Comp
-L Cantaloupe:5_Way_Tactile_Switch SW31
+L Cantaloupe:5_Way_Tactile_Switch SW32
 U 1 1 5F625B45
 P 5800 2700
-F 0 "SW31" H 5800 3115 50  0000 C CNN
+F 0 "SW32" H 5800 3115 50  0000 C CNN
 F 1 "5_Way_Tactile_Switch" H 5800 3024 50  0000 C CNN
 F 2 "Cantaloupe:5-way_Tactile_Switch" H 5800 3150 50  0001 C CNN
@@
 $EndComp
 $Comp
-L Cantaloupe:5_Way_Tactile_Switch SW33
+L Cantaloupe:5_Way_Tactile_Switch SW65
 U 1 1 5F6C5471
 P 5850 6250
-F 0 "SW33" H 5850 6665 50  0000 C CNN
+F 0 "SW65" H 5850 6665 50  0000 C CNN
 F 1 "5_Way_Tactile_Switch_R" H 5850 6574 50  0000 C CNN
 F 2 "Cantaloupe:5-way_Tactile_Switch" H 5850 6700 50  0001 C CNN
@@
 	4450 3150 4450 3200
 $Comp
-L Device:Rotary_Encoder_Switch SW32
+L Device:Rotary_Encoder_Switch SW31
 U 1 1 5FD36B2E
 P 4550 2850
-F 0 "SW32" V 4550 3200 50  0000 C CNN
+F 0 "SW31" V 4550 3200 50  0000 C CNN
 F 1 "Rotary_Encoder_Switch" V 3850 2850 50  0001 C CNN
 F 2 "Rotary_Encoder:RotaryEncoder_Alps_EC11E-Switch_Vertical_H20mm" H 4400 3010 50  0001 C CNN
@@
 	4550 7000 4550 6700
 $Comp
-L Device:Rotary_Encoder_Switch SW66
+L Device:Rotary_Encoder_Switch SW64
 U 1 1 5F63E2D4
 P 4550 6400
-F 0 "SW66" V 4550 6750 50  0000 C CNN
+F 0 "SW64" V 4550 6750 50  0000 C CNN
 F 1 "Rotary_Encoder_Switch" V 3850 6400 50  0001 C CNN
 F 2 "Rotary_Encoder:RotaryEncoder_Alps_EC11E-Switch_Vertical_H20mm" H 4400 6560 50  0001 C CNN
@@
 Connection ~ 2550 5000
 $Comp
-L Cantaloupe:MX-NoLED SW35
+L Cantaloupe:MX-NoLED SW34
 U 1 1 5F63E2B0
 P 3050 4650
-F 0 "SW35" H 3050 4800 50  0000 C CNN
+F 0 "SW34" H 3050 4800 50  0000 C CNN
 F 1 "MX" H 3050 4350 60  0001 C CNN
 F 2 "Cantaloupe:CherryMX_Hotswap_SMK" H 3050 4650 60  0001 C CNN
@@
 	3200 4600 3250 4600
 $Comp
-L Cantaloupe:MX-NoLED SW36
+L Cantaloupe:MX-NoLED SW35
 U 1 1 5F63E2E7
 P 3050 5250
-F 0 "SW36" H 3050 5400 50  0000 C CNN
+F 0 "SW35" H 3050 5400 50  0000 C CNN
 F 1 "MX" H 3050 4950 60  0001 C CNN
 F 2 "Cantaloupe:CherryMX_Hotswap_SMK" H 3050 5250 60  0001 C CNN
@@
 	3200 5200 3250 5200
 $Comp
-L Cantaloupe:MX-NoLED SW37
+L Cantaloupe:MX-NoLED SW36
 U 1 1 5F63E2F4
 P 3050 5850
-F 0 "SW37" H 3050 6000 50  0000 C CNN
+F 0 "SW36" H 3050 6000 50  0000 C CNN
 F 1 "MX" H 3050 5550 60  0001 C CNN
 F 2 "Cantaloupe:CherryMX_Hotswap_SMK" H 3050 5850 60  0001 C CNN
@@
 	3200 5800 3250 5800
 $Comp
-L Cantaloupe:MX-NoLED SW38
+L Cantaloupe:MX-NoLED SW37
 U 1 1 5F63E301
 P 3050 6450
-F 0 "SW38" H 3050 6600 50  0000 C CNN
+F 0 "SW37" H 3050 6600 50  0000 C CNN
 F 1 "MX" H 3050 6150 60  0001 C CNN
 F 2 "Cantaloupe:CherryMX_Hotswap_SMK" H 3050 6450 60  0001 C CNN
@@
 	3200 6400 3250 6400
 $Comp
-L Cantaloupe:MX-NoLED SW39
+L Cantaloupe:MX-NoLED SW38
 U 1 1 5F63E30E
 P 3050 7050
-F 0 "SW39" H 3050 7200 50  0000 C CNN
+F 0 "SW38" H 3050 7200 50  0000 C CNN
 F 1 "MX" H 3050 6750 60  0001 C CNN
 F 2 "Cantaloupe:CherryMX_Hotswap_SMK" H 3050 7050 60  0001 C CNN
@@
 	3000 7400 3550 7400
 $Comp
-L Cantaloupe:MX-NoLED SW40
+L Cantaloupe:MX-NoLED SW39
 U 1 1 5F63E324
 P 2600 4650
-F 0 "SW40" H 2600 4800 50  0000 C CNN
+F 0 "SW39" H 2600 4800 50  0000 C CNN
 F 1 "MX" H 2600 4350 60  0001 C CNN
 F 2 "Cantaloupe:CherryMX_Hotswap_SMK" H 2600 4650 60  0001 C CNN
@@
 	2750 4600 2800 4600
 $Comp
-L Cantaloupe:MX-NoLED SW41
+L Cantaloupe:MX-NoLED SW40
 U 1 1 5F63E332
 P 2600 5250
-F 0 "SW41" H 2600 5400 50  0000 C CNN
+F 0 "SW40" H 2600 5400 50  0000 C CNN
 F 1 "MX" H 2600 4950 60  0001 C CNN
 F 2 "Cantaloupe:CherryMX_Hotswap_SMK" H 2600 5250 60  0001 C CNN
@@
 	2750 5200 2800 5200
 $Comp
-L Cantaloupe:MX-NoLED SW42
+L Cantaloupe:MX-NoLED SW41
 U 1 1 5F63E33F
 P 2600 5850
-F 0 "SW42" H 2600 6000 50  0000 C CNN
+F 0 "SW41" H 2600 6000 50  0000 C CNN
 F 1 "MX" H 2600 5550 60  0001 C CNN
 F 2 "Cantaloupe:CherryMX_Hotswap_SMK" H 2600 5850 60  0001 C CNN
@@
 	2750 5800 2800 5800
 $Comp
-L Cantaloupe:MX-NoLED SW43
+L Cantaloupe:MX-NoLED SW42
 U 1 1 5F63E34C
 P 2600 6450
-F 0 "SW43" H 2600 6600 50  0000 C CNN
+F 0 "SW42" H 2600 6600 50  0000 C CNN
 F 1 "MX" H 2600 6150 60  0001 C CNN
 F 2 "Cantaloupe:CherryMX_Hotswap_SMK" H 2600 6450 60  0001 C CNN
@@
 	2750 6400 2800 6400
 $Comp
-L Cantaloupe:MX-NoLED SW44
+L Cantaloupe:MX-NoLED SW43
 U 1 1 5F63E359
 P 2600 7050
-F 0 "SW44" H 2600 7200 50  0000 C CNN
+F 0 "SW43" H 2600 7200 50  0000 C CNN
 F 1 "MX" H 2600 6750 60  0001 C CNN
 F 2 "Cantaloupe:CherryMX_Hotswap_SMK" H 2600 7050 60  0001 C CNN
@@
 Connection ~ 3000 7400
 $Comp
-L Cantaloupe:MX-NoLED SW45
+L Cantaloupe:MX-NoLED SW44
 U 1 1 5F63E37C
 P 2150 4650
-F 0 "SW45" H 2150 4800 50  0000 C CNN
+F 0 "SW44" H 2150 4800 50  0000 C CNN
 F 1 "MX" H 2150 4350 60  0001 C CNN
 F 2 "Cantaloupe:CherryMX_Hotswap_SMK" H 2150 4650 60  0001 C CNN
@@
 	2300 4600 2350 4600
 $Comp
-L Cantaloupe:MX-NoLED SW46
+L Cantaloupe:MX-NoLED SW45
 U 1 1 5F63E38A
 P 2150 5250
-F 0 "SW46" H 2150 5400 50  0000 C CNN
+F 0 "SW45" H 2150 5400 50  0000 C CNN
 F 1 "MX" H 2150 4950 60  0001 C CNN
 F 2 "Cantaloupe:CherryMX_Hotswap_SMK" H 2150 5250 60  0001 C CNN
@@
 	2300 5200 2350 5200
 $Comp
-L Cantaloupe:MX-NoLED SW47
+L Cantaloupe:MX-NoLED SW46
 U 1 1 5F63E397
 P 2150 5850
-F 0 "SW47" H 2150 6000 50  0000 C CNN
+F 0 "SW46" H 2150 6000 50  0000 C CNN
 F 1 "MX" H 2150 5550 60  0001 C CNN
 F 2 "Cantaloupe:CherryMX_Hotswap_SMK" H 2150 5850 60  0001 C CNN
@@
 	2300 5800 2350 5800
 $Comp
-L Cantaloupe:MX-NoLED SW48
+L Cantaloupe:MX-NoLED SW47
 U 1 1 5F63E3A4
 P 2150 6450
-F 0 "SW48" H 2150 6600 50  0000 C CNN
+F 0 "SW47" H 2150 6600 50  0000 C CNN
 F 1 "MX" H 2150 6150 60  0001 C CNN
 F 2 "Cantaloupe:CherryMX_Hotswap_SMK" H 2150 6450 60  0001 C CNN
@@
 	2300 6400 2350 6400
 $Comp
-L Cantaloupe:MX-NoLED SW49
+L Cantaloupe:MX-NoLED SW48
 U 1 1 5F63E3B1
 P 2150 7050
-F 0 "SW49" H 2150 7200 50  0000 C CNN
+F 0 "SW48" H 2150 7200 50  0000 C CNN
 F 1 "MX" H 2150 6750 60  0001 C CNN
 F 2 "Cantaloupe:CherryMX_Hotswap_SMK" H 2150 7050 60  0001 C CNN
@@
 	2100 7400 2550 7400
 $Comp
-L Cantaloupe:MX-NoLED SW50
+L Cantaloupe:MX-NoLED SW49
 U 1 1 5F63E3D0
 P 1700 4650
-F 0 "SW50" H 1700 4800 50  0000 C CNN
+F 0 "SW49" H 1700 4800 50  0000 C CNN
 F 1 "MX" H 1700 4350 60  0001 C CNN
 F 2 "Cantaloupe:CherryMX_Hotswap_SMK" H 1700 4650 60  0001 C CNN
@@
 	1850 4600 1900 4600
 $Comp
-L Cantaloupe:MX-NoLED SW51
+L Cantaloupe:MX-NoLED SW50
 U 1 1 5F63E3DE
 P 1700 5250
-F 0 "SW51" H 1700 5400 50  0000 C CNN
+F 0 "SW50" H 1700 5400 50  0000 C CNN
 F 1 "MX" H 1700 4950 60  0001 C CNN
 F 2 "Cantaloupe:CherryMX_Hotswap_SMK" H 1700 5250 60  0001 C CNN
@@
 	1850 5200 1900 5200
 $Comp
-L Cantaloupe:MX-NoLED SW52
+L Cantaloupe:MX-NoLED SW51
 U 1 1 5F63E3EB
 P 1700 5850
-F 0 "SW52" H 1700 6000 50  0000 C CNN
+F 0 "SW51" H 1700 6000 50  0000 C CNN
 F 1 "MX" H 1700 5550 60  0001 C CNN
 F 2 "Cantaloupe:CherryMX_Hotswap_SMK" H 1700 5850 60  0001 C CNN
@@
 	1850 5800 1900 5800
 $Comp
-L Cantaloupe:MX-NoLED SW53
+L Cantaloupe:MX-NoLED SW52
 U 1 1 5F63E3F8
 P 1700 6450
-F 0 "SW53" H 1700 6600 50  0000 C CNN
+F 0 "SW52" H 1700 6600 50  0000 C CNN
 F 1 "MX" H 1700 6150 60  0001 C CNN
 F 2 "Cantaloupe:CherryMX_Hotswap_SMK" H 1700 6450 60  0001 C CNN
@@
 $EndComp
 $Comp
-L Cantaloupe:MX-NoLED SW65
+L Cantaloupe:MX-NoLED SW63
 U 1 1 5F63E4BA
 P 800 7050
-F 0 "SW65" H 800 7200 50  0000 C CNN
+F 0 "SW63" H 800 7200 50  0000 C CNN
 F 1 "MX" H 800 6750 60  0001 C CNN
 F 2 "Cantaloupe:CherryMX_Hotswap_SMK" H 800 7050 60  0001 C CNN
@@
 $EndComp
 $Comp
-L Cantaloupe:MX-NoLED SW63
+L Cantaloupe:MX-NoLED SW58
 U 1 1 5F63E493
 P 1250 7050
-F 0 "SW63" H 1250 7200 50  0000 C CNN
+F 0 "SW58" H 1250 7200 50  0000 C CNN
 F 1 "MX" H 1250 6750 60  0001 C CNN
 F 2 "Cantaloupe:CherryMX_Hotswap_SMK" H 1250 7050 60  0001 C CNN
@@
 $EndComp
 $Comp
-L Cantaloupe:MX-NoLED SW58
+L Cantaloupe:MX-NoLED SW53
 U 1 1 5F63E444
 P 1700 7050
-F 0 "SW58" H 1700 7200 50  0000 C CNN
+F 0 "SW53" H 1700 7200 50  0000 C CNN
 F 1 "MX" H 1700 6750 60  0001 C CNN
 F 2 "Cantaloupe:CherryMX_Hotswap_SMK" H 1700 7050 60  0001 C CNN

Commit message: Interconnect changed to C-168688
Changed interconnect footprint to USB C-168688 due to lack of widespread availability of previous part.
Parts:
- J1, J4: footprint Cantaloupe:USB-C-PowerOnly -> Cantaloupe:USB-C-C168688
Changed lines of the file:
@@
 F 0 "J4" H 7907 5167 50  0000 C CNN
 F 1 "USB_C_Receptacle_PD" H 7907 5076 50  0000 C CNN
-F 2 "Cantaloupe:USB-C-PowerOnly" H 7950 4300 50  0001 C CNN
+F 2 "Cantaloupe:USB-C-C168688" H 7950 4300 50  0001 C CNN
 F 3 "https://www.usb.org/sites/default/files/documents/usb_type-c.zip" H 7950 4300 50  0001 C CNN
 	1    7800 4300
@@
 F 0 "J1" H 7857 2267 50  0000 C CNN
 F 1 "USB_C_Receptacle_PD" H 7857 2176 50  0000 C CNN
-F 2 "Cantaloupe:USB-C-PowerOnly" H 7900 1400 50  0001 C CNN
+F 2 "Cantaloupe:USB-C-C168688" H 7900 1400 50  0001 C CNN
 F 3 "https://www.usb.org/sites/default/files/documents/usb_type-c.zip" H 7900 1400 50  0001 C CNN
 	1    7750 1400

Commit message: Updated to V1.1
Parts:
- removed D63, D64, D65, D66, D67, D68, D69, D70: D, Diode_SMD:D_SOD-123, symbol Device:D_Small
- removed J1, J4: USB_C_Receptacle_PD, Cantaloupe:USB-C-C168688, symbol Cantaloupe:USB_C_Receptacle_PD
- removed J2, J5: Bat, Cantaloupe:Battery_Solder_Points, symbol Connector_Generic:Conn_01x02
- removed J3, J6: OLED, Cantaloupe:PinHeader_1x04_P2.54mm_Vertical_No_Silk, symbol Connector_Generic:Conn_01x04
- removed R1, R2: 10k, Resistor_SMD:R_0603_1608Metric_Pad1.05x0.95mm_HandSolder, symbol Device:R_Small
- removed SW31, SW64: Rotary_Encoder_Switch, Rotary_Encoder:RotaryEncoder_Alps_EC11E-Switch_Vertical_H20mm, symbol Device:Rotary_Encoder_Switch
- removed SW32: 5_Way_Tactile_Switch, Cantaloupe:5-way_Tactile_Switch, symbol Cantaloupe:5_Way_Tactile_Switch
- removed SW65: 5_Way_Tactile_Switch_R, Cantaloupe:5-way_Tactile_Switch, symbol Cantaloupe:5_Way_Tactile_Switch
- added J1, J4: OLED, Cantaloupe:PinHeader_1x04_P2.54mm_Vertical_No_Silk, symbol Connector_Generic:Conn_01x04
- added J2: Interconnect, Cantaloupe:USB-C_C168688, symbol Connector:USB_C_Receptacle_USB2.0
- added J3: ICSP, Connector_PinHeader_2.54mm:PinHeader_2x03_P2.54mm_Vertical, symbol Connector_Generic:Conn_02x03_Odd_Even
- added J5: Interconnect_R, Cantaloupe:USB-C_C168688, symbol Connector:USB_C_Receptacle_USB2.0
- added J6: ICSP_R, Connector_PinHeader_2.54mm:PinHeader_2x03_P2.54mm_Vertical, symbol Connector_Generic:Conn_02x03_Odd_Even
- added J7: BAT_CON_TOG, Cantaloupe:Battery_Solder_Points, symbol Connector_Generic:Conn_01x02
- added J8: BAT_CON_R, Cantaloupe:Battery_Solder_Points, symbol Connector_Generic:Conn_01x02
- added J9: BAT_CON, Cantaloupe:Battery_Solder_Points, symbol Connector_Generic:Conn_01x02
- added SW31, SW64: MX, Cantaloupe:CherryMX_Hotswap_SMK, symbol Cantaloupe:MX-NoLED
- added SW32: Encoder, Rotary_Encoder:RotaryEncoder_Alps_EC11E-Switch_Vertical_H20mm, symbol Device:Rotary_Encoder_Switch
- added SW65: Encoder_R, Rotary_Encoder:RotaryEncoder_Alps_EC11E-Switch_Vertical_H20mm, symbol Device:Rotary_Encoder_Switch
- added SW67: BAT_TOG, Cantaloupe:Switch_MSK-22D18, symbol Switch:SW_Push_DPDT
- added SW68: BAT_TOG_R, Cantaloupe:Switch_MSK-22D18, symbol Switch:SW_Push_DPDT
Connections:
- net labels added: RAW_R, ROT_A, ROT_A_R, ROT_B, ROT_B_R
- net labels removed: GND2, ROTA, ROTA_R, ROTB, ROTB_R
- wire segments 218 -> 241
- no-connect marks 4 -> 14
Other:
- moved on the sheet: D1, D10, D11, D12, D13, D14, D15, D16, D17, D18, D19, D2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
