File: Hardware/Cantaloupe.sch (KiCad schematic (older format))
At the start: 141 parts, among them J1 BAT_CON, J2 OLED, J3 Interconnect, J4 ICSP, J5 BAT_CON_TOG, J6 OLED, J7 Interconnect_R, J8 ICSP_R, J9 BAT_CON_R, SW1 MX, SW10 MX, SW11 MX, SW12 MX, SW13 MX, SW14 MX, SW15 MX, SW16 MX, SW17 MX, SW18 MX, SW19 MX, SW2 MX, SW20 MX, SW21 MX, SW22 MX, SW23 MX, SW24 MX, SW25 MX, SW26 MX, SW27 MX, SW28 MX, SW29 MX, SW3 MX, SW30 MX, SW31 Reset, SW32 5_Way, SW33 BAT_TOG, SW34 Encoder, SW35 MX, SW36 MX, SW37 MX, SW38 MX, SW39 MX, SW4 MX, SW40 MX, SW41 MX, SW42 MX, SW43 MX, SW44 MX, SW45 MX, SW46 MX, SW47 MX, SW48 MX, SW49 MX, SW5 MX, SW50 MX, SW51 MX, SW52 MX, SW53 MX, SW54 MX, SW55 MX, SW56 MX, SW57 MX, SW58 MX, SW59 MX, SW6 MX, SW60 MX, SW61 MX, SW62 MX, SW63 MX, SW64 MX, SW65 Reset, SW66 5_Way_R, SW67 Encoder_R, SW68 BAT_TOG_R, SW7 MX, SW8 MX, SW9 MX, U1 ProMicro, U2 ProMicro

Commit message: Updated to V1.2
Parts:
- removed SW32: 5_Way, Cantaloupe:Switch_5-way-tactile, symbol Cantaloupe:Switch_5-Way-Tactile
- removed SW66: 5_Way_R, Cantaloupe:Switch_5-way-tactile, symbol Cantaloupe:Switch_5-Way-Tactile
- added SW31, SW65: MX, Cantaloupe:HYBRID-MX_ALPS_SMK-1U, symbol Cantaloupe:MX-NoLED
- D1, D10, D11, D12, D13, D14, D15, D16, D17, D18, D19, D2, D20, D21, D22, D23, D24, D25, D26, D27, D28, D29, D3, D30, D31, D32, D33, D34, D35, D36, D37, D38, D39, D4, D40, D41, D42, D43, D44, D45, D46, D47, D48, D49, D5, D50, D51, D52, D53, D54, D55, D56, D57, D58, D59, D6, D60, D61, D62, D7, D8, D9: footprint Diode_SMD:D_SOD-123 -> Cantaloupe:D_Hybrid_SOD123_DO35
- SW1, SW10, SW11, SW12, SW13, SW14, SW15, SW16, SW17, SW18, SW19, SW2, SW20, SW21, SW22, SW23, SW24, SW25, SW26, SW27, SW28, SW29, SW3, SW30, SW35, SW36, SW37, SW38, SW39, SW4, SW40, SW41, SW42, SW43, SW44, SW45, SW46, SW47, SW48, SW49, SW5, SW50, SW51, SW52, SW53, SW54, SW55, SW56, SW57, SW58, SW59, SW6, SW60, SW61, SW62, SW63, SW64, SW7, SW8, SW9: footprint Cantaloupe:MX-1U-Hotswap -> Cantaloupe:HYBRID-MX_ALPS_SMK-1U
- renumbered J2 to J1, J3 to J2, J4 to J3, J1 to J4, J9 to J5, J5 to J9, SW34 to SW32, SW31 to SW33, SW33 to SW34, SW67 to SW66, SW65 to SW67
Connections:
- net COL0: now also U1.19 (A2/PF5); no longer U1.7 (4/PD4)
- net COL0_R: now also U2.7 (4/PD4); no longer U2.19 (A2/PF5)
- net COL1: now also U1.18 (A1/PF6); no longer U1.8 (5/PC6)
- net COL1_R: now also U2.8 (5/PC6); no longer U2.18 (A1/PF6)
- net COL2: now also U1.17 (A0/PF7); no longer U1.9 (6/PD7)
- net COL2_R: now also U2.9 (6/PD7); no longer U2.17 (A0/PF7)
- net COL3: now also U1.16 (15/PB1); no longer U1.10 (7/PE6)
- net COL3_R: now also U2.10 (7/PE6); no longer U2.16 (15/PB1)
- net COL4: now also U1.15 (14/PB3); no longer U1.11 (8/PB4)
- net COL4_R: now also U2.11 (8/PB4); no longer U2.15 (14/PB3)
- net COL5: now also U1.14 (16/PB2); no longer U1.12 (9/PB5)
- net COL5_R: now also U2.12 (9/PB5); no longer U2.14 (16/PB2)
- net GND1: no longer J1.1 (Pin_1), J2.A1 (GND), J2.A12 (GND), J2.B1 (GND), J2.B12 (GND), J2.S1 (SHIELD), J3.6 (Pin_6), SW32.C, SW33.2
- net GND3: now also U2.4 (GND); no longer J5.1 (Pin_1), U2.23 (GND)
- net PERIPH: now also SW32.S2, U1.1 (TX0/PD3), SW31.1 (COL); no longer D31.2 (A), U1.19 (A2/PF5)
- net PERIPH_R: now also SW66.S2, U2.20 (A3/PF4), SW65.1 (COL); no longer D62.2 (A), U2.1 (TX0/PD3)
- net ROT_A: now also U1.7 (4/PD4); no longer U1.18 (A1/PF6)
- net ROT_A_R: now also U2.19 (A2/PF5); no longer U2.7 (4/PD4)
- net ROT_B: now also U1.8 (5/PC6); no longer U1.17 (A0/PF7)
- net ROT_B_R: now also U2.18 (A1/PF6); no longer U2.8 (5/PC6)
- net ROW0: now also U1.20 (A3/PF4); no longer U1.1 (TX0/PD3)
- net ROW0_R: now also U2.1 (TX0/PD3); no longer U2.20 (A3/PF4)
- net ROW1: now also U1.12 (9/PB5); no longer SW32.S2, U1.13 (10/PB6)
- net ROW1_R: now also U2.14 (16/PB2); no longer U2.12 (9/PB5)
- net ROW2: now also U1.11 (8/PB4); no longer U1.14 (16/PB2)
- net ROW2_R: now also U2.15 (14/PB3); no longer U2.11 (8/PB4)
- net ROW3: now also U1.10 (7/PE6); no longer U1.15 (14/PB3)
- net ROW3_R: now also U2.16 (15/PB1); no longer SW66.S2, U2.10 (7/PE6)
- net ROW4: now also D31.1 (K), U1.9 (6/PD7); no longer U1.16 (15/PB1)
- net ROW4_R: now also D62.1 (K), U2.17 (A0/PF7); no longer U2.9 (6/PD7)
- net at J4.2 (Pin_2): now also SW34.3 (C), SW34.6 (C); no longer U1.24 (RAW)
- net GND2: now reaches U1.4 (GND)
- net GND2: now also J1.1 (Pin_1), J2.A1 (GND), J2.A12 (GND), J2.B1 (GND), J2.B12 (GND), J2.S1 (SHIELD), J3.6 (Pin_6), SW32.C, SW33.2
- net at SW32.S1: now also D31.2 (A), SW31.2 (ROW); no longer D31.1 (K)
- net RAW: now reaches SW34.2 (B), SW34.5 (B)
- net RAW: now also U1.24 (RAW); no longer J9.1 (Pin_1)
- net at SW68.1 (A), SW68.4 (A): now also J9.2 (Pin_2); no longer J5.2 (Pin_2)
- net at SW66.S1: now also D62.2 (A), SW65.2 (ROW); no longer D62.1 (K)
- net RAW_R: no longer names the net of SW68.2 (B), SW68.5 (B)
- net RAW_R: now also J9.1 (Pin_1); no longer U2.24 (RAW)
- new net: J5.1 (Pin_1), U2.23 (GND)
- new net: J5.2 (Pin_2), U2.24 (RAW)
- no-connect marks 14 -> 12
Other:
- moved on the sheet: D1, D10, D11, D12, D13, D14, D15, D16, D17, D18, D19, D2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

Commit message: Changed USB C connector to normal from mid-mount
Parts:
- J2, J7: footprint Cantaloupe:USB-C_C168688 -> Connector_USB:USB_C_Receptacle_HRO_TYPE-C-31-M-12
Connections:
- net GND3 is gone; now on net GND2: J6.1 (Pin_1), J7.A1 (GND), J7.A12 (GND), J7.B1 (GND), J7.B12 (GND), J7.S1 (SHIELD), J8.6 (Pin_6), SW66.C, SW67.2, U2.4 (GND)
- net GND1: now also J1.1 (Pin_1), J2.A1 (GND), J2.A12 (GND), J2.B1 (GND), J2.B12 (GND), J2.S1 (SHIELD), J3.6 (Pin_6), SW32.C, SW33.2, U1.4 (GND)
- net GND2: now also J5.1 (Pin_1), U2.23 (GND); no longer J1.1 (Pin_1), J2.A1 (GND), J2.A12 (GND), J2.B1 (GND), J2.B12 (GND), J2.S1 (SHIELD), J3.6 (Pin_6), SW32.C, SW33.2, U1.4 (GND)
Changed lines of the file:
@@
 Wire Wire Line
 	1400 7350 1400 7550
-$Comp
-L power:GND3 #PWR012
-U 1 1 6020CBB8
-P 1400 7550
-F 0 "#PWR012" H 1400 7300 50  0001 C CNN
-F 1 "GND3" H 1405 7377 50  0000 C CNN
-F 2 "" H 1400 7550 50  0001 C CNN
-F 3 "" H 1400 7550 50  0001 C CNN
-	1    1400 7550
-	1    0    0    -1
-$EndComp
 Connection ~ 2450 3200
 Wire Wire Line
@@
 F 0 "J2" H 7957 2717 50  0000 C CNN
 F 1 "Interconnect" H 7957 2626 50  0000 C CNN
-F 2 "Cantaloupe:USB-C_C168688" H 8000 1850 50  0001 C CNN
+F 2 "Connector_USB:USB_C_Receptacle_HRO_TYPE-C-31-M-12" H 8000 1850 50  0001 C CNN
 F 3 "" H 8000 1850 50  0001 C CNN
 	1    7850 1850
@@
 F 0 "J7" H 7907 6267 50  0000 C CNN
 F 1 "Interconnect_R" H 7907 6176 50  0000 C CNN
-F 2 "Cantaloupe:USB-C_C168688" H 7950 5400 50  0001 C CNN
+F 2 "Connector_USB:USB_C_Receptacle_HRO_TYPE-C-31-M-12" H 7950 5400 50  0001 C CNN
 F 3 "" H 7950 5400 50  0001 C CNN
 	1    7800 5400
@@
 	1    0    0    -1
 $EndComp
-$Comp
-L power:GND3 #PWR021
-U 1 1 6078345A
-P 7650 6300
-F 0 "#PWR021" H 7650 6050 50  0001 C CNN
-F 1 "GND3" H 7655 6127 50  0000 C CNN
-F 2 "" H 7650 6300 50  0001 C CNN
-F 3 "" H 7650 6300 50  0001 C CNN
-	1    7650 6300
-	1    0    0    -1
-$EndComp
-Wire Wire Line
-	7800 6300 7650 6300
-Connection ~ 7650 6300
-Wire Wire Line
-	7650 6300 7500 6300
 Wire Wire Line
 	8450 1750 8450 1850
@@
 NoConn ~ 8450 1450
 $Comp
-L power:GND3 #PWR016
-U 1 1 5FCAA71A
-P 9550 4650
-F 0 "#PWR016" H 9550 4400 50  0001 C CNN
-F 1 "GND3" H 9555 4477 50  0000 C CNN
-F 2 "" H 9550 4650 50  0001 C CNN
-F 3 "" H 9550 4650 50  0001 C CNN
-	1    9550 4650
-	1    0    0    -1
-$EndComp
-$Comp
 L power:VDD #PWR013
 U 1 1 5FCAA161
@@
 Text GLabel 9350 5300 0    50   Input ~ 0
 RESET_R
-$Comp
-L power:GND3 #PWR018
-U 1 1 5F795E0A
-P 9750 5300
-F 0 "#PWR018" H 9750 5050 50  0001 C CNN
-F 1 "GND3" H 9755 5127 50  0000 C CNN
-F 2 "" H 9750 5300 50  0001 C CNN
-F 3 "" H 9750 5300 50  0001 C CNN
-	1    9750 5300
-	1    0    0    -1
-$EndComp
 Text GLabel 5800 4600 2    50   Input ~ 0
 RESET_R
@@
 Wire Wire Line
 	6200 4350 6200 4700
-NoConn ~ 4400 4600
-$Comp
-L power:GND3 #PWR015
-U 1 1 5F77703F
-P 3950 4700
-F 0 "#PWR015" H 3950 4450 50  0001 C CNN
-F 1 "GND3" H 3955 4527 50  0000 C CNN
-F 2 "" H 3950 4700 50  0001 C CNN
-F 3 "" H 3950 4700 50  0001 C CNN
-	1    3950 4700
-	1    0    0    -1
-$EndComp
 Wire Wire Line
 	9450 950  9250 950
@@
 F 3 "" H 9800 6050 50  0001 C CNN
 	1    9800 6050
-	1    0    0    -1
-$EndComp
-$Comp
-L power:GND3 #PWR020
-U 1 1 5FA25D01
-P 9800 6250
-F 0 "#PWR020" H 9800 6000 50  0001 C CNN
-F 1 "GND3" H 9805 6077 50  0000 C CNN
-F 2 "" H 9800 6250 50  0001 C CNN
-F 3 "" H 9800 6250 50  0001 C CNN
-	1    9800 6250
 	1    0    0    -1
 $EndComp
@@
 Connection ~ 2200 3550
 Connection ~ 2400 3750
-$Comp
-L power:GND2 #PWR0101
-U 1 1 603BD7A0
+Wire Wire Line
+	4450 1200 4150 1200
+Wire Wire Line
+	4150 1200 4150 1100
+Wire Wire Line
+	4150 1100 4050 1100
+NoConn ~ 5850 2000
+Wire Wire Line
+	5800 4500 6400 4500
+Wire Wire Line
+	4400 4700 3950 4700
+Wire Wire Line
+	6400 4600 6400 4500
+Connection ~ 6400 4500
+Wire Wire Line
+	6400 4500 6500 4500
+Wire Wire Line
+	7550 2750 7700 2750
+$Comp
+L power:GND1 #PWR0101
+U 1 1 5FB37F40
+P 7700 2750
+F 0 "#PWR0101" H 7700 2500 50  0001 C CNN
+F 1 "GND1" H 7705 2577 50  0000 C CNN
+F 2 "" H 7700 2750 50  0001 C CNN
+F 3 "" H 7700 2750 50  0001 C CNN
+	1    7700 2750
+	1    0    0    -1
+$EndComp
+Connection ~ 7700 2750
+Wire Wire Line
+	7700 2750 7850 2750
+$Comp
+L power:GND1 #PWR0102
+U 1 1 5FB38560
+P 9650 1850
+F 0 "#PWR0102" H 9650 1600 50  0001 C CNN
+F 1 "GND1" H 9655 1677 50  0000 C CNN
+F 2 "" H 9650 1850 50  0001 C CNN
+F 3 "" H 9650 1850 50  0001 C CNN
+	1    9650 1850
+	1    0    0    -1
+$EndComp
+$Comp
+L power:GND1 #PWR0103
+U 1 1 5FB38EF9
+P 9450 1150
+F 0 "#PWR0103" H 9450 900 50  0001 C CNN
+F 1 "GND1" H 9455 977 50  0000 C CNN
+F 2 "" H 9450 1150 50  0001 C CNN
+F 3 "" H 9450 1150 50  0001 C CNN
+	1    9450 1150
+	1    0    0    -1
+$EndComp
+$Comp
+L power:GND1 #PWR0104
+U 1 1 5FB3930B
+P 9750 2700
+F 0 "#PWR0104" H 9750 2450 50  0001 C CNN
+F 1 "GND1" H 9755 2527 50  0000 C CNN
+F 2 "" H 9750 2700 50  0001 C CNN
+F 3 "" H 9750 2700 50  0001 C CNN
+	1    9750 2700
+	1    0    0    -1
+$EndComp
+$Comp
+L power:GND1 #PWR0105
+U 1 1 5FB3970C
+P 4050 1100
+F 0 "#PWR0105" H 4050 850 50  0001 C CNN
+F 1 "GND1" H 4055 927 50  0000 C CNN
+F 2 "" H 4050 1100 50  0001 C CNN
+F 3 "" H 4050 1100 50  0001 C CNN
+	1    4050 1100
+	1    0    0    -1
+$EndComp
+$Comp
+L power:GND1 #PWR0106
+U 1 1 5FB49731
 P 1300 3800
-F 0 "#PWR0101" H 1300 3550 50  0001 C CNN
-F 1 "GND2" H 1305 3627 50  0000 C CNN
+F 0 "#PWR0106" H 1300 3550 50  0001 C CNN
+F 1 "GND1" H 1305 3627 50  0000 C CNN
 F 2 "" H 1300 3800 50  0001 C CNN
 F 3 "" H 1300 3800 50  0001 C CNN
@@
 $EndComp
 $Comp
-L power:GND2 #PWR0102
-U 1 1 603CD687
-P 7700 2750
-F 0 "#PWR0102" H 7700 2500 50  0001 C CNN
-F 1 "GND2" H 7705 2577 50  0000 C CNN
-F 2 "" H 7700 2750 50  0001 C CNN
-F 3 "" H 7700 2750 50  0001 C CNN
-	1    7700 2750
-	1    0    0    -1
-$EndComp
-Wire Wire Line
-	7550 2750 7700 2750
-Connection ~ 7700 2750
-Wire Wire Line
-	7700 2750 7850 2750
-$Comp
-L power:GND2 #PWR0103
-U 1 1 603DD2AF
-P 9750 2700
-F 0 "#PWR0103" H 9750 2450 50  0001 C CNN
-F 1 "GND2" H 9755 2527 50  0000 C CNN
-F 2 "" H 9750 2700 50  0001 C CNN
-F 3 "" H 9750 2700 50  0001 C CNN
-	1    9750 2700
-	1    0    0    -1
-$EndComp
-$Comp
-L power:GND2 #PWR0104
-U 1 1 603DD777
-P 9650 1850
-F 0 "#PWR0104" H 9650 1600 50  0001 C CNN
-F 1 "GND2" H 9655 1677 50  0000 C CNN
-F 2 "" H 9650 1850 50  0001 C CNN
-F 3 "" H 9650 1850 50  0001 C CNN
-	1    9650 1850
-	1    0    0    -1
-$EndComp
-$Comp
-L power:GND2 #PWR0105
-U 1 1 603DDB5D
-P 9450 1150
-F 0 "#PWR0105" H 9450 900 50  0001 C CNN
-F 1 "GND2" H 9455 977 50  0000 C CNN
-F 2 "" H 9450 1150 50  0001 C CNN
-F 3 "" H 9450 1150 50  0001 C CNN
-	1    9450 1150
-	1    0    0    -1
-$EndComp
-$Comp
-L power:GND2 #PWR0106
-U 1 1 603DE5C2
-P 4050 1100
-F 0 "#PWR0106" H 4050 850 50  0001 C CNN
-F 1 "GND2" H 4055 927 50  0000 C CNN
-F 2 "" H 4050 1100 50  0001 C CNN
-F 3 "" H 4050 1100 50  0001 C CNN
-	1    4050 1100
-	1    0    0    -1
-$EndComp
-Wire Wire Line
-	4450 1200 4150 1200
-Wire Wire Line
-	4150 1200 4150 1100
-Wire Wire Line
-	4150 1100 4050 1100
-NoConn ~ 5850 2000
-Wire Wire Line
-	5800 4500 6500 4500
-Wire Wire Line
-	4400 4700 3950 4700
+L power:GND2 #PWR0107
+U 1 1 5FB5A117
+P 9550 4650
+F 0 "#PWR0107" H 9550 4400 50  0001 C CNN
+F 1 "GND2" H 9555 4477 50  0000 C CNN
+F 2 "" H 9550 4650 50  0001 C CNN
+F 3 "" H 9550 4650 50  0001 C CNN
+	1    9550 4650
+	1    0    0    -1
+$EndComp
+$Comp
+L power:GND2 #PWR0108
+U 1 1 5FB6AFE2
+P 9800 6250
+F 0 "#PWR0108" H 9800 6000 50  0001 C CNN
+F 1 "GND2" H 9805 6077 50  0000 C CNN
+F 2 "" H 9800 6250 50  0001 C CNN
+F 3 "" H 9800 6250 50  0001 C CNN
+	1    9800 6250
+	1    0    0    -1
+$EndComp
+$Comp
+L power:GND2 #PWR0109
+U 1 1 5FB7B029
+P 7650 6300
+F 0 "#PWR0109" H 7650 6050 50  0001 C CNN
+F 1 "GND2" H 7655 6127 50  0000 C CNN
+F 2 "" H 7650 6300 50  0001 C CNN
+F 3 "" H 7650 6300 50  0001 C CNN
+	1    7650 6300
+	1    0    0    -1
+$EndComp
+Connection ~ 7650 6300
+Wire Wire Line
+	7650 6300 7800 6300
+Wire Wire Line
+	7500 6300 7650 6300
+$Comp
+L power:GND2 #PWR0110
+U 1 1 5FB9ABF8
+P 6400 4600
+F 0 "#PWR0110" H 6400 4350 50  0001 C CNN
+F 1 "GND2" H 6405 4427 50  0000 C CNN
+F 2 "" H 6400 4600 50  0001 C CNN
+F 3 "" H 6400 4600 50  0001 C CNN
+	1    6400 4600
+	1    0    0    -1
+$EndComp
+$Comp
+L power:GND2 #PWR0111
+U 1 1 5FBAAC9E
+P 3950 4700
+F 0 "#PWR0111" H 3950 4450 50  0001 C CNN
+F 1 "GND2" H 3955 4527 50  0000 C CNN
+F 2 "" H 3950 4700 50  0001 C CNN
+F 3 "" H 3950 4700 50  0001 C CNN
+	1    3950 4700
+	1    0    0    -1
+$EndComp
+$Comp
+L power:GND2 #PWR0112
+U 1 1 5FBBB468
+P 1400 7550
+F 0 "#PWR0112" H 1400 7300 50  0001 C CNN
+F 1 "GND2" H 1405 7377 50  0000 C CNN
+F 2 "" H 1400 7550 50  0001 C CNN
+F 3 "" H 1400 7550 50  0001 C CNN
+	1    1400 7550
+	1    0    0    -1
+$EndComp
+$Comp
+L power:GND2 #PWR0113
+U 1 1 5FBCCE7E
+P 9750 5300
+F 0 "#PWR0113" H 9750 5050 50  0001 C CNN
+F 1 "GND2" H 9755 5127 50  0000 C CNN
+F 2 "" H 9750 5300 50  0001 C CNN
+F 3 "" H 9750 5300 50  0001 C CNN
+	1    9750 5300
+	1    0    0    -1
+$EndComp
+NoConn ~ 4400 4600
 $EndSCHEMATC

Commit message: Updated to V1.3.
Parts:
- added SW31, SW32, SW67, SW68: MX, Cantaloupe:HYBRID-MX_ALPS-2U-ReversedStabilizers-NoLED, symbol Cantaloupe:SW_Push_Small
- SW1, SW10, SW11, SW12, SW13, SW14, SW15, SW16, SW17, SW18, SW19, SW2, SW20, SW21, SW22, SW23, SW24, SW25, SW26, SW27, SW28, SW29, SW3, SW30, SW4, SW5, SW6, SW7, SW8, SW9: footprint Cantaloupe:HYBRID-MX_ALPS_SMK-1U -> Cantaloupe:HYBRID-MX_ALPS-1U-NoLED; symbol Cantaloupe:MX-NoLED -> Cantaloupe:SW_Push_Small
- SW34: renamed from SW31; footprint Cantaloupe:HYBRID-MX_ALPS_SMK-1U -> Cantaloupe:HYBRID-MX_ALPS-1U-NoLED; symbol Cantaloupe:MX-NoLED -> Cantaloupe:SW_Push_Small
- SW37: renamed from SW35; footprint Cantaloupe:HYBRID-MX_ALPS_SMK-1U -> Cantaloupe:HYBRID-MX_ALPS-1U-NoLED; symbol Cantaloupe:MX-NoLED -> Cantaloupe:SW_Push_Small
- SW38: renamed from SW36; footprint Cantaloupe:HYBRID-MX_ALPS_SMK-1U -> Cantaloupe:HYBRID-MX_ALPS-1U-NoLED; symbol Cantaloupe:MX-NoLED -> Cantaloupe:SW_Push_Small
- SW39: renamed from SW37; footprint Cantaloupe:HYBRID-MX_ALPS_SMK-1U -> Cantaloupe:HYBRID-MX_ALPS-1U-NoLED; symbol Cantaloupe:MX-NoLED -> Cantaloupe:SW_Push_Small
- SW40: renamed from SW38; footprint Cantaloupe:HYBRID-MX_ALPS_SMK-1U -> Cantaloupe:HYBRID-MX_ALPS-1U-NoLED; symbol Cantaloupe:MX-NoLED -> Cantaloupe:SW_Push_Small
- SW41: renamed from SW39; footprint Cantaloupe:HYBRID-MX_ALPS_SMK-1U -> Cantaloupe:HYBRID-MX_ALPS-1U-NoLED; symbol Cantaloupe:MX-NoLED -> Cantaloupe:SW_Push_Small
- SW42: renamed from SW40; footprint Cantaloupe:HYBRID-MX_ALPS_SMK-1U -> Cantaloupe:HYBRID-MX_ALPS-1U-NoLED; symbol Cantaloupe:MX-NoLED -> Cantaloupe:SW_Push_Small
- SW43: renamed from SW41; footprint Cantaloupe:HYBRID-MX_ALPS_SMK-1U -> Cantaloupe:HYBRID-MX_ALPS-1U-NoLED; symbol Cantaloupe:MX-NoLED -> Cantaloupe:SW_Push_Small
- SW44: renamed from SW42; footprint Cantaloupe:HYBRID-MX_ALPS_SMK-1U -> Cantaloupe:HYBRID-MX_ALPS-1U-NoLED; symbol Cantaloupe:MX-NoLED -> Cantaloupe:SW_Push_Small
- SW45: renamed from SW43; footprint Cantaloupe:HYBRID-MX_ALPS_SMK-1U -> Cantaloupe:HYBRID-MX_ALPS-1U-NoLED; symbol Cantaloupe:MX-NoLED -> Cantaloupe:SW_Push_Small
- SW46: renamed from SW44; footprint Cantaloupe:HYBRID-MX_ALPS_SMK-1U -> Cantaloupe:HYBRID-MX_ALPS-1U-NoLED; symbol Cantaloupe:MX-NoLED -> Cantaloupe:SW_Push_Small
- SW47: renamed from SW45; footprint Cantaloupe:HYBRID-MX_ALPS_SMK-1U -> Cantaloupe:HYBRID-MX_ALPS-1U-NoLED; symbol Cantaloupe:MX-NoLED -> Cantaloupe:SW_Push_Small
- SW48: renamed from SW46; footprint Cantaloupe:HYBRID-MX_ALPS_SMK-1U -> Cantaloupe:HYBRID-MX_ALPS-1U-NoLED; symbol Cantaloupe:MX-NoLED -> Cantaloupe:SW_Push_Small
- SW49: renamed from SW47; footprint Cantaloupe:HYBRID-MX_ALPS_SMK-1U -> Cantaloupe:HYBRID-MX_ALPS-1U-NoLED; symbol Cantaloupe:MX-NoLED -> Cantaloupe:SW_Push_Small
- SW50: renamed from SW48; footprint Cantaloupe:HYBRID-MX_ALPS_SMK-1U -> Cantaloupe:HYBRID-MX_ALPS-1U-NoLED; symbol Cantaloupe:MX-NoLED -> Cantaloupe:SW_Push_Small
- SW51: renamed from SW49; footprint Cantaloupe:HYBRID-MX_ALPS_SMK-1U -> Cantaloupe:HYBRID-MX_ALPS-1U-NoLED; symbol Cantaloupe:MX-NoLED -> Cantaloupe:SW_Push_Small
- SW52: renamed from SW50; footprint Cantaloupe:HYBRID-MX_ALPS_SMK-1U -> Cantaloupe:HYBRID-MX_ALPS-1U-NoLED; symbol Cantaloupe:MX-NoLED -> Cantaloupe:SW_Push_Small
- SW53: renamed from SW51; footprint Cantaloupe:HYBRID-MX_ALPS_SMK-1U -> Cantaloupe:HYBRID-MX_ALPS-1U-NoLED; symbol Cantaloupe:MX-NoLED -> Cantaloupe:SW_Push_Small
- SW54: renamed from SW52; footprint Cantaloupe:HYBRID-MX_ALPS_SMK-1U -> Cantaloupe:HYBRID-MX_ALPS-1U-NoLED; symbol Cantaloupe:MX-NoLED -> Cantaloupe:SW_Push_Small
- SW55: renamed from SW53; footprint Cantaloupe:HYBRID-MX_ALPS_SMK-1U -> Cantaloupe:HYBRID-MX_ALPS-1U-NoLED; symbol Cantaloupe:MX-NoLED -> Cantaloupe:SW_Push_Small
- SW56: renamed from SW54; footprint Cantaloupe:HYBRID-MX_ALPS_SMK-1U -> Cantaloupe:HYBRID-MX_ALPS-1U-NoLED; symbol Cantaloupe:MX-NoLED -> Cantaloupe:SW_Push_Small
- SW57: renamed from SW55; footprint Cantaloupe:HYBRID-MX_ALPS_SMK-1U -> Cantaloupe:HYBRID-MX_ALPS-1U-NoLED; symbol Cantaloupe:MX-NoLED -> Cantaloupe:SW_Push_Small
- SW58: renamed from SW56; footprint Cantaloupe:HYBRID-MX_ALPS_SMK-1U -> Cantaloupe:HYBRID-MX_ALPS-1U-NoLED; symbol Cantaloupe:MX-NoLED -> Cantaloupe:SW_Push_Small
- SW59: renamed from SW57; footprint Cantaloupe:HYBRID-MX_ALPS_SMK-1U -> Cantaloupe:HYBRID-MX_ALPS-1U-NoLED; symbol Cantaloupe:MX-NoLED -> Cantaloupe:SW_Push_Small
- SW60: renamed from SW58; footprint Cantaloupe:HYBRID-MX_ALPS_SMK-1U -> Cantaloupe:HYBRID-MX_ALPS-1U-NoLED; symbol Cantaloupe:MX-NoLED -> Cantaloupe:SW_Push_Small
- SW61: renamed from SW59; footprint Cantaloupe:HYBRID-MX_ALPS_SMK-1U -> Cantaloupe:HYBRID-MX_ALPS-1U-NoLED; symbol Cantaloupe:MX-NoLED -> Cantaloupe:SW_Push_Small
- SW62: renamed from SW60; footprint Cantaloupe:HYBRID-MX_ALPS_SMK-1U -> Cantaloupe:HYBRID-MX_ALPS-1U-NoLED; symbol Cantaloupe:MX-NoLED -> Cantaloupe:SW_Push_Small
- SW63: renamed from SW61; footprint Cantaloupe:HYBRID-MX_ALPS_SMK-1U -> Cantaloupe:HYBRID-MX_ALPS-1U-NoLED; symbol Cantaloupe:MX-NoLED -> Cantaloupe:SW_Push_Small
- SW64: renamed from SW62; footprint Cantaloupe:HYBRID-MX_ALPS_SMK-1U -> Cantaloupe:HYBRID-MX_ALPS-1U-NoLED; symbol Cantaloupe:MX-NoLED -> Cantaloupe:SW_Push_Small
- SW65: renamed from SW63; footprint Cantaloupe:HYBRID-MX_ALPS_SMK-1U -> Cantaloupe:HYBRID-MX_ALPS-1U-NoLED; symbol Cantaloupe:MX-NoLED -> Cantaloupe:SW_Push_Small
- SW66: renamed from SW64; footprint Cantaloupe:HYBRID-MX_ALPS_SMK-1U -> Cantaloupe:HYBRID-MX_ALPS-1U-NoLED; symbol Cantaloupe:MX-NoLED -> Cantaloupe:SW_Push_Small
- SW70: renamed from SW65; footprint Cantaloupe:HYBRID-MX_ALPS_SMK-1U -> Cantaloupe:HYBRID-MX_ALPS-1U-NoLED; symbol Cantaloupe:MX-NoLED -> Cantaloupe:SW_Push_Small
- renumbered SW32 to SW33, SW33 to SW35, SW34 to SW36, SW66 to SW69, SW67 to SW71, SW68 to SW72
Connections:
- net COL0: now also SW31.1
- net COL0_R: now also SW67.1
- net PERIPH: now also U1.8 (5/PC6), SW32.1; no longer U1.1 (TX0/PD3)
- net PERIPH_R: now also U2.18 (A1/PF6), SW68.1; no longer U2.20 (A3/PF4)
- net ROT_A_R: now also U2.20 (A3/PF4); no longer U2.19 (A2/PF5)
- net ROT_B: now also U1.1 (TX0/PD3); no longer U1.8 (5/PC6)
- net ROT_B_R: now also U2.19 (A2/PF5); no longer U2.18 (A1/PF6)
- net at D25.2 (A), SW25.2: now also SW31.2
- net at D31.2 (A), SW33.S1, SW34.2: now also SW32.2
- net at D61.2 (A), SW66.2: now also SW67.2
- net at D62.2 (A), SW69.S1, SW70.2: now also SW68.2
Other:
- moved on the sheet: D1, D10, D11, D12, D13, D14, D15, D16, D17, D18, D19, D2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
