File: Hardware/Cantaloupe.kicad_pcb (KiCad board)
At the start: 2 copper layers, 287.3 x 117 mm, 169 parts, among them J1 BAT_CON, J2 OLED, J3 Interconnect, J4 ICSP, J5 BAT_CON_TOG, J6 OLED, J7 Interconnect_R, J8 ICSP_R, J9 BAT_CON_R, SW1 MX, SW10 MX, SW11 MX, SW12 MX, SW13 MX, SW14 MX, SW15 MX, SW16 MX, SW17 MX, SW18 MX, SW19 MX, SW2 MX, SW20 MX, SW21 MX, SW22 MX, SW23 MX, SW24 MX, SW25 MX, SW26 MX, SW27 MX, SW28 MX, SW29 MX, SW3 MX, SW30 MX, SW31 Reset, SW32 5_Way, SW33 BAT_TOG, SW34 Encoder, SW35 MX, SW36 MX, SW37 MX, SW38 MX, SW39 MX, SW4 MX, SW40 MX, SW41 MX, SW42 MX, SW43 MX, SW44 MX, SW45 MX, SW46 MX, SW47 MX, SW48 MX, SW49 MX, SW5 MX, SW50 MX, SW51 MX, SW52 MX, SW53 MX, SW54 MX, SW55 MX, SW56 MX, SW57 MX, SW58 MX, SW59 MX, SW6 MX, SW60 MX, SW61 MX, SW62 MX, SW63 MX, SW64 MX, SW65 Reset, SW66 5_Way_R, SW67 Encoder_R, SW68 BAT_TOG_R, SW7 MX, SW8 MX, SW9 MX, U1 ProMicro, U2 ProMicro

Commit message: Fixed position of RHS screw hole and wiring of rotary encoder switch, added QMK firmware.
Parts:
- moved REF** 1.50 mm to (98.4, 57.1)
Connections:
- SW34 pad S2: PERIPH -> ROW1
- SW67 pad S2: PERIPH_R -> ROW3_R
Routing:
- net PERIPH_R: track 124.5 -> 108.4 mm
- net ROW1: track 186.5 -> 188.5 mm
- net ROW3_R: track 234.7 -> 236.6 mm
Changed lines of the file:
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@@
     (thickness 1.6)
     (drawings 74)
-    (tracks 1151)
+    (tracks 1153)
     (zones 0)
     (modules 169)
@@
       (net 94 ROT_A))
     (pad S2 thru_hole circle (at 7 -2.5 60) (size 2 2) (drill 1) (layers *.Cu *.Mask)
-      (net 106 PERIPH))
+      (net 2 ROW1))
     (model ${KISYS3DMOD}/Rotary_Encoder.3dshapes/RotaryEncoder_Alps_EC11E-Switch_Vertical_H20mm.wrl
       (at (xyz 0 0 0))
@@
   )
   (module MountingHole:MountingHole_2.2mm_M2_Pad (layer F.Cu)
-    (at 98.424701 58.584931)
+    (at 98.424701 57.084877)
     (descr "Mounting Hole 2.2mm, M2")
     (tags "mounting hole 2.2mm m2")
@@
       (net 98 ROT_A_R))
     (pad S2 thru_hole circle (at 7 -2.5 120) (size 2 2) (drill 1) (layers *.Cu *.Mask)
-      (net 109 PERIPH_R))
+      (net 42 ROW3_R))
     (model ${KISYS3DMOD}/Rotary_Encoder.3dshapes/RotaryEncoder_Alps_EC11E-Switch_Vertical_H20mm.wrl
       (at (xyz 0 0 0))
@@
   (segment (start 309.555951 71.353924) (end 309.562499 71.347376) (width 0.25) (layer B.Cu) (net 2))
   (segment (start 309.555951 73.24964) (end 309.555951 71.353924) (width 0.25) (layer B.Cu) (net 2))
+  (segment (start 327.258141 114.032953) (end 328.403686 112.887408) (width 0.25) (layer F.Cu) (net 2))
+  (segment (start 326.887828 114.032953) (end 327.258141 114.032953) (width 0.25) (layer F.Cu) (net 2))
   (segment (start 232.421869 50.584878) (end 233.362499 50.584878) (width 0.25) (layer B.Cu) (net 3))
   (segment (start 231.267001 49.43001) (end 232.421869 50.584878) (width 0.25) (layer B.Cu) (net 3))
@@
   (segment (start 80.630952 112.978852) (end 80.630952 112.060667) (width 0.25) (layer B.Cu) (net 42))
   (segment (start 80.54265 113.067154) (end 80.630952 112.978852) (width 0.25) (layer B.Cu) (net 42))
+  (segment (start 58.025029 115.621604) (end 57.790887 115.387462) (width 0.25) (layer F.Cu) (net 42))
+  (segment (start 58.025029 117.273007) (end 58.025029 115.621604) (width 0.25) (layer F.Cu) (net 42))
   (segment (start 191.146869 50.584878) (end 192.087499 50.584878) (width 0.25) (layer B.Cu) (net 43))
   (segment (start 189.992001 45.654877) (end 189.992001 49.43001) (width 0.25) (layer B.Cu) (net 43))
@@
   (segment (start 311.605951 111.29041) (end 311.605951 52.64964) (width 0.25) (layer F.Cu) (net 105))
   (segment (start 311.605951 52.64964) (end 311.958213 52.297378) (width 0.25) (layer F.Cu) (net 105))
-  (segment (start 316.887086 112.887408) (end 328.403686 112.887408) (width 0.25) (layer B.Cu) (net 106))
-  (segment (start 314.093719 112.887408) (end 316.887086 112.887408) (width 0.25) (layer B.Cu) (net 106))
-  (segment (start 312.737551 73.06804) (end 312.737551 111.53124) (width 0.25) (layer B.Cu) (net 106))
-  (segment (start 336.185096 52.599973) (end 336.185096 66.602434) (width 0.25) (layer B.Cu) (net 106))
-  (segment (start 312.737551 111.53124) (end 314.093719 112.887408) (width 0.25) (layer B.Cu) (net 106))
-  (segment (start 336.185096 66.602434) (end 333.122734 69.664796) (width 0.25) (layer B.Cu) (net 106))
-  (segment (start 333.122734 69.664796) (end 316.140795 69.664796) (width 0.25) (layer B.Cu) (net 106))
-  (segment (start 332.73375 49.148627) (end 336.185096 52.599973) (width 0.25) (layer B.Cu) (net 106))
-  (segment (start 316.140795 69.664796) (end 312.737551 73.06804) (width 0.25) (layer B.Cu) (net 106))
-  (segment (start 328.403686 122.932177) (end 332.367826 126.896317) (width 0.25) (layer B.Cu) (net 106))
-  (segment (start 328.403686 112.887408) (end 328.403686 122.932177) (width 0.25) (layer B.Cu) (net 106))
-  (segment (start 332.508333 117.277953) (end 332.508333 115.612889) (width 0.25) (layer B.Cu) (net 107) (status 30))
+  (segment (start 336.185096 52.599973) (end 332.73375 49.148627) (width 0.25) (layer B.Cu) (net 106))
+  (segment (start 336.185096 66.602434) (end 336.185096 52.599973) (width 0.25) (layer B.Cu) (net 106))
+  (segment (start 333.122734 69.664796) (end 336.185096 66.602434) (width 0.25) (layer B.Cu) (net 106))
+  (segment (start 312.737551 73.06804) (end 316.140795 69.664796) (width 0.25) (layer B.Cu) (net 106))
+  (segment (start 328.380952 122.909443) (end 328.380952 115.625639) (width 0.25) (layer B.Cu) (net 106))
+  (segment (start 328.380952 115.625639) (end 327.838276 115.082963) (width 0.25) (layer B.Cu) (net 106))
+  (segment (start 332.367826 126.896317) (end 328.380952 122.909443) (width 0.25) (layer B.Cu) (net 106))
+  (segment (start 327.838276 115.082963) (end 313.224947 115.082963) (width 0.25) (layer B.Cu) (net 106))
+  (segment (start 316.140795 69.664796) (end 333.122734 69.664796) (width 0.25) (layer B.Cu) (net 106))
+  (segment (start 312.737551 114.595567) (end 312.737551 73.06804) (width 0.25) (layer B.Cu) (net 106))
+  (segment (start 313.224947 115.082963) (end 312.737551 114.595567) (width 0.25) (layer B.Cu) (net 106))
   (segment (start 332.508333 115.612889) (end 332.733814 115.387408) (width 0.25) (layer B.Cu) (net 107) (status 30))
   (segment (start 334.767827 123.288432) (end 334.017826 124.038433) (width 0.25) (layer B.Cu) (net 107))
   (segment (start 332.508333 117.277953) (end 334.767827 119.537447) (width 0.25) (layer B.Cu) (net 107))
   (segment (start 334.767827 119.537447) (end 334.767827 123.288432) (width 0.25) (layer B.Cu) (net 107))
+  (segment (start 332.508333 115.612889) (end 332.733814 115.387408) (width 0.25) (layer F.Cu) (net 107))
+  (segment (start 332.508333 117.277953) (end 332.508333 115.612889) (width 0.25) (layer F.Cu) (net 107))
   (segment (start 192.087201 53.884931) (end 173.037201 53.884931) (width 0.25) (layer B.Cu) (net 108))
   (segment (start 173.037201 53.884931) (end 160.312555 53.884931) (width 0.25) (layer B.Cu) (net 108))
@@
   (segment (start 98.25816 52.297431) (end 96.837201 52.297431) (width 0.25) (layer B.Cu) (net 108))
   (segment (start 95.179702 74.673391) (end 95.179702 111.475889) (width 0.25) (layer F.Cu) (net 108))
-  (segment (start 62.013716 119.610291) (end 57.790887 115.387462) (width 0.25) (layer B.Cu) (net 109))
-  (segment (start 71.253607 119.610291) (end 62.013716 119.610291) (width 0.25) (layer B.Cu) (net 109))
-  (segment (start 71.905028 118.95887) (end 71.253607 119.610291) (width 0.25) (layer B.Cu) (net 109))
   (segment (start 72.56258 118.95887) (end 71.905028 118.95887) (width 0.25) (layer B.Cu) (net 109))
   (segment (start 77.905901 113.615549) (end 72.56258 118.95887) (width 0.25) (layer B.Cu) (net 109))
@@
   (segment (start 54.327105 38.128486) (end 54.327105 66.589636) (width 0.25) (layer B.Cu) (net 109))
   (segment (start 54.327105 66.589636) (end 57.402268 69.664799) (width 0.25) (layer B.Cu) (net 109))
-  (segment (start 62.121015 112.887462) (end 62.504989 112.887462) (width 0.25) (layer B.Cu) (net 110) (status 30))
-  (segment (start 62.504989 112.887462) (end 63.645534 114.028007) (width 0.25) (layer B.Cu) (net 110) (status 30))
   (segment (start 68.182049 114.028007) (end 70.255028 116.100986) (width 0.25) (layer B.Cu) (net 110))
   (segment (start 63.645534 114.028007) (end 68.182049 114.028007) (width 0.25) (layer B.Cu) (net 110))
+  (segment (start 62.504989 112.887462) (end 63.645534 114.028007) (width 0.25) (layer B.Cu) (net 110))
+  (segment (start 62.121015 112.887462) (end 62.504989 112.887462) (width 0.25) (layer B.Cu) (net 110))
   (segment (start 337.34375 36.448627) (end 332.97531 36.448627) (width 1.7526) (layer F.Cu) (net 111) (status 30))
   (segment (start 337.34375 36.448627) (end 332.97531 36.448627) (width 1.7526) (layer B.Cu) (net 111) (status 30))

Commit message: Updated to V1.2
Parts:
- removed the J1 at (337.3, 39.0)
- removed the J5 at (309.6, 33.7)
- removed the REF** at (174.6, 60.3)
- removed the REF** at (98.4, 57.1)
- removed the REF** at (117.5, 112.6)
- removed the REF** at (174.6, 117.4)
- removed the REF** at (312.2, 121.5)
- removed the REF** at (273.1, 112.6)
- removed the REF** at (292.1, 57.1)
- removed the REF** at (215.9, 117.4)
- removed the REF** at (215.9, 60.3)
- removed the SW32 at (327.1, 120.2)
- removed the SW66 at (63.5, 120.2)
- added J4: BAT_CON, Cantaloupe:Battery_Solder_Points, B.Cu at (312.9, 39.1)
- added J9: BAT_CON_TOG, Cantaloupe:Battery_Solder_Points, F.Cu at (78.3, 33.8)
- added REF**: MountingHole_2.2mm_M2_Pad, MountingHole:MountingHole_2.2mm_M2_Pad, F.Cu at (174.6, 60.3)
- added REF**: MountingHole_2.2mm_M2_Pad, MountingHole:MountingHole_2.2mm_M2_Pad, F.Cu at (98.4, 57.1)
- added REF**: MountingHole_2.2mm_M2_Pad, MountingHole:MountingHole_2.2mm_M2_Pad, F.Cu at (117.5, 112.7)
- added REF**: MountingHole_2.2mm_M2_Pad, MountingHole:MountingHole_2.2mm_M2_Pad, F.Cu at (174.6, 117.5)
- added REF**: MountingHole_2.2mm_M2_Pad, MountingHole:MountingHole_2.2mm_M2_Pad, F.Cu at (312.2, 121.5)
- added REF**: MountingHole_2.2mm_M2_Pad, MountingHole:MountingHole_2.2mm_M2_Pad, F.Cu at (273.0, 112.7)
- added REF**: MountingHole_2.2mm_M2_Pad, MountingHole:MountingHole_2.2mm_M2_Pad, F.Cu at (292.1, 57.1)
- added REF**: MountingHole_2.2mm_M2_Pad, MountingHole:MountingHole_2.2mm_M2_Pad, F.Cu at (215.9, 117.5)
- added REF**: MountingHole_2.2mm_M2_Pad, MountingHole:MountingHole_2.2mm_M2_Pad, F.Cu at (215.9, 60.3)
- added SW31: MX, Cantaloupe:HYBRID-MX_ALPS_SMK-1U, F.Cu at (327.1, 120.3)
- added SW65: MX, Cantaloupe:HYBRID-MX_ALPS_SMK-1U, F.Cu at (63.5, 120.3)
- D1, D10, D11, D12, D13, D14, D15, D16, D17, D18, D19, D2, D20, D21, D22, D23, D24, D25, D26, D27, D28, D29, D3, D30, D31, D32, D33, D34, D35, D36, D37, D38, D39, D4, D40, D41, D42, D43, D44, D45, D46, D47, D48, D49, D5, D50, D51, D52, D53, D54, D55, D56, D57, D58, D59, D6, D60, D61, D62, D7, D8, D9: footprint Diode_SMD:D_SOD-123 -> Cantaloupe:D_Hybrid_SOD123_DO35
- J2: renamed from J3; moved to F.Cu
- J5: renamed from J9; moved to B.Cu
- J7: moved to F.Cu
- SW1, SW10, SW11, SW12, SW13, SW14, SW15, SW16, SW17, SW18, SW19, SW2, SW20, SW21, SW22, SW23, SW24, SW25, SW26, SW27, SW28, SW29, SW3, SW30, SW35, SW36, SW37, SW38, SW39, SW4, SW40, SW41, SW42, SW43, SW44, SW45, SW46, SW47, SW48, SW49, SW5, SW50, SW51, SW52, SW53, SW54, SW55, SW56, SW57, SW58, SW59, SW6, SW60, SW61, SW62, SW63, SW64, SW7, SW8, SW9: footprint Cantaloupe:MX-1U-Hotswap -> Cantaloupe:HYBRID-MX_ALPS_SMK-1U
- U1, U2: moved to B.Cu
- moved J5 24.5 mm to (53.2, 39.1), turned to 0 degrees
- moved D12 1.52 mm to (309.6, 68.2)
- moved D14 1.52 mm to (233.4, 88.8)
- moved D15 1.52 mm to (252.4, 84.0)
- moved D16 1.52 mm to (271.5, 80.1)
- moved D17 1.52 mm to (290.5, 84.0)
- moved D18 1.52 mm to (309.6, 87.2)
- moved D19 1.52 mm to (214.3, 107.9)
- moved D20 1.52 mm to (233.4, 107.9)
- moved D21 1.52 mm to (252.4, 103.1)
- moved D22 1.52 mm to (271.5, 99.1)
- moved D25 1.52 mm to (214.3, 126.9)
- moved D26 1.52 mm to (233.4, 126.9)
- moved D36 1.52 mm to (173.0, 50.7)
- moved D37 1.52 mm to (192.1, 50.7)
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- renumbered J2 to J1, J4 to J3, SW34 to SW32, SW31 to SW33, SW33 to SW34, SW67 to SW66, SW65 to SW67
Connections:
- D31 pad 1: Net-(D31-Pad1) -> ROW4
- D31 pad 2: PERIPH -> Net-(D31-Pad2)
- D62 pad 1: Net-(D62-Pad1) -> ROW4_R
- D62 pad 2: PERIPH_R -> Net-(D62-Pad2)
- J1 pad 1: GND1 -> GND2
- J2 pad A1: GND1 -> GND2
- J2 pad S1: GND1 -> GND2
- J3 pad 6: GND1 -> GND2
- J5 pad 1: GND3 -> Net-(J5-Pad1)
- J5 pad 2: Net-(J9-Pad2) -> Net-(J5-Pad2)
- SW32 pad C: GND1 -> GND2
- SW32 pad S1: Net-(D31-Pad1) -> Net-(D31-Pad2)
- SW32 pad S2: ROW1 -> PERIPH
- SW33 pad 2: GND1 -> GND2
- SW34 pad 2: Net-(J5-Pad1) -> RAW
- SW34 pad 5: Net-(J5-Pad1) -> RAW
- SW66 pad S1: Net-(D62-Pad1) -> Net-(D62-Pad2)
- SW66 pad S2: ROW3_R -> PERIPH_R
- SW68 pad 2: RAW_R -> Net-(J9-Pad1)
- SW68 pad 5: RAW_R -> Net-(J9-Pad1)
- U1 pad 1: ROW0 -> PERIPH
- U1 pad 10: COL3 -> ROW3
- U1 pad 11: COL4 -> ROW2
- U1 pad 12: COL5 -> ROW1
- U1 pad 13: ROW1 -> Net-(U1-Pad13)
- U1 pad 14: ROW2 -> COL5
- U1 pad 15: ROW3 -> COL4
- U1 pad 16: ROW4 -> COL3
- U1 pad 17: ROT_B -> COL2
- U1 pad 18: ROT_A -> COL1
- U1 pad 19: PERIPH -> COL0
- U1 pad 20: Net-(U1-Pad20) -> ROW0
- U1 pad 24: Net-(J1-Pad2) -> RAW
- U1 pad 4: Net-(U1-Pad4) -> GND2
- U1 pad 7: COL0 -> ROT_A
- U1 pad 8: COL1 -> ROT_B
- U1 pad 9: COL2 -> ROW4
- U2 pad 1: PERIPH_R -> ROW0_R
- U2 pad 10: ROW3_R -> COL3_R
- U2 pad 11: ROW2_R -> COL4_R
- U2 pad 12: ROW1_R -> COL5_R
- U2 pad 14: COL5_R -> ROW1_R
- U2 pad 15: COL4_R -> ROW2_R
- U2 pad 16: COL3_R -> ROW3_R
- U2 pad 17: COL2_R -> ROW4_R
- U2 pad 18: COL1_R -> ROT_B_R
- U2 pad 19: COL0_R -> ROT_A_R
- U2 pad 20: ROW0_R -> PERIPH_R
- U2 pad 23: GND3 -> Net-(J5-Pad1)
- U2 pad 24: RAW_R -> Net-(J5-Pad2)
- U2 pad 4: Net-(U2-Pad4) -> GND3
- U2 pad 7: ROT_A_R -> COL0_R
- U2 pad 8: ROT_B_R -> COL1_R
- U2 pad 9: ROW4_R -> COL2_R
Routing:
- net GND1: track 154.4 -> 4.61 mm, vias 2 -> 0
- net GND2: track 0.00 -> 137.9 mm
- net ROW0_R: track 231.9 -> 149.4 mm, vias 3 -> 0
- net ROW0: track 206.5 -> 124.5 mm, vias 1 -> 0
- net ROW1_R: track 221.6 -> 160.7 mm, vias 3 -> 0
- net ROW1: track 188.5 -> 142.4 mm, vias 1 -> 0
- net ROW2_R: track 221.0 -> 182.7 mm, vias 3 -> 0
- net COL3_R: track 239.6 -> 207.1 mm, vias 6 -> 1
- net ROW3_R: track 236.6 -> 204.6 mm, vias 1 -> 0
- net COL5: track 143.0 -> 115.0 mm, vias 5 -> 0
- net COL4_R: track 202.0 -> 174.4 mm, vias 6 -> 1
- net COL3: track 173.1 -> 151.4 mm, vias 5 -> 0
- net COL4: track 157.3 -> 135.8 mm, vias 5 -> 0
- net COL2: track 180.2 -> 160.2 mm, vias 5 -> 0
- net COL5_R: track 164.3 -> 145.6 mm, vias 5 -> 0
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Other:
- board text added: "Cantaloupe V1.2 Aria"
- board text removed: "Cantaloupe V1.1 Aria"
- board text removed: "JLCJLCJLCJLC"

Commit message: Changed USB C connector to normal from mid-mount
Parts:
- removed the REF** at (196.8, 88.9)
- removed the REF** at (196.8, 127.0)
- removed the REF** at (193.7, 127.0)
- removed the REF** at (193.7, 88.9)
- removed the REF** at (196.8, 50.8)
- removed the REF** at (193.7, 50.8)
- J2, J7: footprint Cantaloupe:USB-C_C168688 -> Connector_USB:USB_C_Receptacle_HRO_TYPE-C-31-M-12
- moved J3 5.68 mm to (334.5, 109.2), turned to 0 degrees
- moved J2 3.03 mm to (336.9, 82.2), turned to 90 degrees
- moved J7 3.00 mm to (53.6, 82.2), turned to 270 degrees
Connections:
- J1 pad 1: GND2 -> GND1
- J2 pad A1: GND2 -> GND1
- J2 pad S1: GND2 -> GND1
- J3 pad 6: GND2 -> GND1
- J5 pad 1: Net-(J5-Pad1) -> GND2
- J6 pad 1: GND3 -> GND2
- J7 pad A1: GND3 -> GND2
- J7 pad S1: GND3 -> GND2
- J8 pad 6: GND3 -> GND2
- SW32 pad C: GND2 -> GND1
- SW33 pad 2: GND2 -> GND1
- SW66 pad C: GND3 -> GND2
- SW67 pad 2: GND3 -> GND2
- U1 pad 4: GND2 -> GND1
- U2 pad 23: Net-(J5-Pad1) -> GND2
- U2 pad 4: GND3 -> GND2
Routing:
- net GND3: track 174.1 -> 0.00 mm
- net GND1: track 4.61 -> 116.7 mm
- net GND2: track 137.9 -> 154.2 mm
- net RESET: track 83.8 -> 74.1 mm, vias 2 -> 0
- net ROT_B: track 103.7 -> 113.0 mm
- net VCC: track 78.4 -> 85.3 mm, vias 0 -> 1
- net ROW3: track 220.1 -> 213.3 mm, vias 1 -> 0
- net ROT_B_R: track 104.7 -> 99.0 mm
- net PERIPH_R: track 114.6 -> 108.9 mm
- net ROT_A_R: track 111.5 -> 105.8 mm
- net ROW4_R: track 246.9 -> 241.9 mm
- net Net-(J5-Pad1): track 4.61 -> 0.00 mm
- net COL3_R: track 207.1 -> 211.3 mm
- net RESET_R: track 74.2 -> 77.5 mm, vias 1 -> 0
- net COL2_R: track 151.9 -> 155.2 mm
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Other:
- outline, holes or cut-outs redrawn

Commit message: Updated to V1.3.
Parts:
- removed the REF** at (312.2, 121.5)
- removed the REF** at (273.0, 112.7)
- removed the REF** at (292.1, 57.1)
- removed the REF** at (215.9, 117.5)
- removed the REF** at (215.9, 60.3)
- removed the REF** at (174.6, 60.3)
- removed the REF** at (98.4, 57.1)
- removed the REF** at (117.5, 112.7)
- removed the REF** at (174.6, 117.5)
- added REF**: MountingHole_4.3mm_M4, MountingHole:MountingHole_4.3mm_M4, F.Cu at (312.2, 121.5)
- added REF**: MountingHole_4.3mm_M4, MountingHole:MountingHole_4.3mm_M4, F.Cu at (273.1, 112.7)
- added REF**: MountingHole_4.3mm_M4, MountingHole:MountingHole_4.3mm_M4, F.Cu at (292.1, 57.1)
- added REF**: MountingHole_4.3mm_M4, MountingHole:MountingHole_4.3mm_M4, F.Cu at (215.9, 117.5)
- added REF**: MountingHole_4.3mm_M4, MountingHole:MountingHole_4.3mm_M4, F.Cu at (215.9, 60.3)
- added REF**: MountingHole_4.3mm_M4, MountingHole:MountingHole_4.3mm_M4, F.Cu at (174.6, 60.3)
- added REF**: MountingHole_4.3mm_M4, MountingHole:MountingHole_4.3mm_M4, F.Cu at (98.4, 57.1)
- added REF**: MountingHole_4.3mm_M4, MountingHole:MountingHole_4.3mm_M4, F.Cu at (117.5, 112.7)
- added REF**: MountingHole_4.3mm_M4, MountingHole:MountingHole_4.3mm_M4, F.Cu at (174.6, 117.5)
- added SW31: MX, Cantaloupe:HYBRID-MX_ALPS-2U-ReversedStabilizers-NoLED, F.Cu at (215.9, 127.0)
- added SW32: MX, Cantaloupe:HYBRID-MX_ALPS-2U-ReversedStabilizers-NoLED, F.Cu at (322.3, 128.5)
- added SW67: MX, Cantaloupe:HYBRID-MX_ALPS-2U-ReversedStabilizers-NoLED, F.Cu at (174.6, 127.0)
- added SW68: MX, Cantaloupe:HYBRID-MX_ALPS-2U-ReversedStabilizers-NoLED, F.Cu at (68.2, 128.5)
- REF** (x5): value MountingHole_2.2mm_M2_Pad -> MountingHole_4.3mm_M4; footprint MountingHole:MountingHole_2.2mm_M2_Pad -> MountingHole:MountingHole_4.3mm_M4
- SW1, SW10, SW11, SW12, SW13, SW14, SW15, SW16, SW17, SW18, SW19, SW2, SW20, SW21, SW22, SW23, SW24, SW25, SW26, SW27, SW28, SW29, SW3, SW30, SW4, SW5, SW6, SW7, SW8, SW9: footprint Cantaloupe:HYBRID-MX_ALPS_SMK-1U -> Cantaloupe:HYBRID-MX_ALPS-1U-NoLED
- SW34: renamed from SW31; footprint Cantaloupe:HYBRID-MX_ALPS_SMK-1U -> Cantaloupe:HYBRID-MX_ALPS-1U-NoLED
- SW37: renamed from SW35; footprint Cantaloupe:HYBRID-MX_ALPS_SMK-1U -> Cantaloupe:HYBRID-MX_ALPS-1U-NoLED
- SW38: renamed from SW36; footprint Cantaloupe:HYBRID-MX_ALPS_SMK-1U -> Cantaloupe:HYBRID-MX_ALPS-1U-NoLED
- SW39: renamed from SW37; footprint Cantaloupe:HYBRID-MX_ALPS_SMK-1U -> Cantaloupe:HYBRID-MX_ALPS-1U-NoLED
- SW40: renamed from SW38; footprint Cantaloupe:HYBRID-MX_ALPS_SMK-1U -> Cantaloupe:HYBRID-MX_ALPS-1U-NoLED
- SW41: renamed from SW39; footprint Cantaloupe:HYBRID-MX_ALPS_SMK-1U -> Cantaloupe:HYBRID-MX_ALPS-1U-NoLED
- SW42: renamed from SW40; footprint Cantaloupe:HYBRID-MX_ALPS_SMK-1U -> Cantaloupe:HYBRID-MX_ALPS-1U-NoLED
- SW43: renamed from SW41; footprint Cantaloupe:HYBRID-MX_ALPS_SMK-1U -> Cantaloupe:HYBRID-MX_ALPS-1U-NoLED
- SW44: renamed from SW42; footprint Cantaloupe:HYBRID-MX_ALPS_SMK-1U -> Cantaloupe:HYBRID-MX_ALPS-1U-NoLED
- SW45: renamed from SW43; footprint Cantaloupe:HYBRID-MX_ALPS_SMK-1U -> Cantaloupe:HYBRID-MX_ALPS-1U-NoLED
- SW46: renamed from SW44; footprint Cantaloupe:HYBRID-MX_ALPS_SMK-1U -> Cantaloupe:HYBRID-MX_ALPS-1U-NoLED
- SW47: renamed from SW45; footprint Cantaloupe:HYBRID-MX_ALPS_SMK-1U -> Cantaloupe:HYBRID-MX_ALPS-1U-NoLED
- SW48: renamed from SW46; footprint Cantaloupe:HYBRID-MX_ALPS_SMK-1U -> Cantaloupe:HYBRID-MX_ALPS-1U-NoLED
- SW49: renamed from SW47; footprint Cantaloupe:HYBRID-MX_ALPS_SMK-1U -> Cantaloupe:HYBRID-MX_ALPS-1U-NoLED
- SW50: renamed from SW48; footprint Cantaloupe:HYBRID-MX_ALPS_SMK-1U -> Cantaloupe:HYBRID-MX_ALPS-1U-NoLED
- SW51: renamed from SW49; footprint Cantaloupe:HYBRID-MX_ALPS_SMK-1U -> Cantaloupe:HYBRID-MX_ALPS-1U-NoLED
- SW52: renamed from SW50; footprint Cantaloupe:HYBRID-MX_ALPS_SMK-1U -> Cantaloupe:HYBRID-MX_ALPS-1U-NoLED
- SW53: renamed from SW51; footprint Cantaloupe:HYBRID-MX_ALPS_SMK-1U -> Cantaloupe:HYBRID-MX_ALPS-1U-NoLED
- SW54: renamed from SW52; footprint Cantaloupe:HYBRID-MX_ALPS_SMK-1U -> Cantaloupe:HYBRID-MX_ALPS-1U-NoLED
- SW55: renamed from SW53; footprint Cantaloupe:HYBRID-MX_ALPS_SMK-1U -> Cantaloupe:HYBRID-MX_ALPS-1U-NoLED
- SW56: renamed from SW54; footprint Cantaloupe:HYBRID-MX_ALPS_SMK-1U -> Cantaloupe:HYBRID-MX_ALPS-1U-NoLED
- SW57: renamed from SW55; footprint Cantaloupe:HYBRID-MX_ALPS_SMK-1U -> Cantaloupe:HYBRID-MX_ALPS-1U-NoLED
- SW58: renamed from SW56; footprint Cantaloupe:HYBRID-MX_ALPS_SMK-1U -> Cantaloupe:HYBRID-MX_ALPS-1U-NoLED
- SW59: renamed from SW57; footprint Cantaloupe:HYBRID-MX_ALPS_SMK-1U -> Cantaloupe:HYBRID-MX_ALPS-1U-NoLED
- SW60: renamed from SW58; footprint Cantaloupe:HYBRID-MX_ALPS_SMK-1U -> Cantaloupe:HYBRID-MX_ALPS-1U-NoLED
- SW61: renamed from SW59; footprint Cantaloupe:HYBRID-MX_ALPS_SMK-1U -> Cantaloupe:HYBRID-MX_ALPS-1U-NoLED
- SW62: renamed from SW60; footprint Cantaloupe:HYBRID-MX_ALPS_SMK-1U -> Cantaloupe:HYBRID-MX_ALPS-1U-NoLED
- SW63: renamed from SW61; footprint Cantaloupe:HYBRID-MX_ALPS_SMK-1U -> Cantaloupe:HYBRID-MX_ALPS-1U-NoLED
- SW64: renamed from SW62; footprint Cantaloupe:HYBRID-MX_ALPS_SMK-1U -> Cantaloupe:HYBRID-MX_ALPS-1U-NoLED
- SW65: renamed from SW63; footprint Cantaloupe:HYBRID-MX_ALPS_SMK-1U -> Cantaloupe:HYBRID-MX_ALPS-1U-NoLED
- SW66: renamed from SW64; footprint Cantaloupe:HYBRID-MX_ALPS_SMK-1U -> Cantaloupe:HYBRID-MX_ALPS-1U-NoLED
- SW70: renamed from SW65; footprint Cantaloupe:HYBRID-MX_ALPS_SMK-1U -> Cantaloupe:HYBRID-MX_ALPS-1U-NoLED
- moved D31 19.2 mm to (314.7, 124.1)
- moved D56 18.5 mm to (61.3, 132.5), turned to 300 degrees
- moved D62 9.56 mm to (75.8, 124.1), turned to 300 degrees
- moved D30 9.52 mm to (329.2, 132.5), turned to 240 degrees
- moved D25 8.37 mm to (216.7, 134.9), turned to 180 degrees
- moved D60 8.16 mm to (174.5, 134.9), turned to 180 degrees
- moved J2 0.90 mm to (337.8, 82.2)
- moved J7 0.87 mm to (52.7, 82.2)
- moved REF** 0.20 mm to (70.9, 92.7)
- moved REF** 0.20 mm to (319.6, 92.7)
- turned SW33 to 240 degrees
- turned SW34 to 150 degrees
- turned SW69 to 300 degrees
- turned SW70 to 210 degrees
- turned SW61 to 210 degrees
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- renumbered SW32 to SW33, SW33 to SW35, SW34 to SW36, SW66 to SW69, SW67 to SW71, SW68 to SW72
Connections:
- U1 pad 1: PERIPH -> ROT_B
- U1 pad 8: ROT_B -> PERIPH
- U2 pad 18: ROT_B_R -> PERIPH_R
- U2 pad 19: ROT_A_R -> ROT_B_R
- U2 pad 20: PERIPH_R -> ROT_A_R
Routing:
- net Net-(D25-Pad2): track 7.11 -> 27.3 mm
- net ROW4_R: track 241.9 -> 259.6 mm
- net ROW4: track 279.4 -> 263.2 mm
- net GND1: track 116.7 -> 101.8 mm
- net COL0_R: track 195.0 -> 209.3 mm
- net GND2: track 154.2 -> 140.7 mm
- net Net-(D62-Pad2): track 9.79 -> 22.7 mm
- net Net-(D61-Pad2): track 7.11 -> 18.6 mm
- net Net-(D30-Pad2): track 7.11 -> 18.0 mm
- net COL0: track 202.1 -> 212.1 mm
- net COL5_R: track 146.6 -> 156.1 mm
- net PERIPH_R: track 108.9 -> 99.9 mm
- net Net-(D60-Pad2): track 7.11 -> 15.7 mm
- net Net-(D56-Pad2): track 7.11 -> 14.9 mm
- net COL5: track 115.0 -> 122.5 mm
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Other:
- board size 287.3 x 117 mm -> 289.7 x 117 mm
- board text added: "Cantaloupe V1.3 Aria"
- board text removed: "Cantaloupe V1.2 Aria"
