File: Hardware/Cantaloupe.kicad_pcb (KiCad board)
At the start: 2 copper layers, 289.7 x 117 mm, 161 parts, among them J1 OLED, J2 Interconnect, J3 ICSP, J4 BAT_CON, J5 BAT_CON_R, J6 OLED, J7 Interconnect_R, J8 ICSP_R, J9 BAT_CON_TOG, SW1 MX, SW10 MX, SW11 MX, SW12 MX, SW13 MX, SW14 MX, SW15 MX, SW16 MX, SW17 MX, SW18 MX, SW19 MX, SW2 MX, SW20 MX, SW21 MX, SW22 MX, SW23 MX, SW24 MX, SW25 MX, SW26 MX, SW27 MX, SW28 MX, SW29 MX, SW3 MX, SW30 MX, SW31 MX, SW32 MX, SW33 Encoder, SW34 MX, SW35 Reset, SW36 BAT_TOG, SW37 MX, SW38 MX, SW39 MX, SW4 MX, SW40 MX, SW41 MX, SW42 MX, SW43 MX, SW44 MX, SW45 MX, SW46 MX, SW47 MX, SW48 MX, SW49 MX, SW5 MX, SW50 MX, SW51 MX, SW52 MX, SW53 MX, SW54 MX, SW55 MX, SW56 MX, SW57 MX, SW58 MX, SW59 MX, SW6 MX, SW60 MX, SW61 MX, SW62 MX, SW63 MX, SW64 MX, SW65 MX, SW66 MX, SW67 MX, SW68 MX, SW69 Encoder_R, SW7 MX, SW70 MX, SW71 Reset, SW72 BAT_TOG_R, SW8 MX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

Commit message: Added proper OLED support.
Parts:
- added REF**: MountingHole_2.2mm_M2, MountingHole:MountingHole_2.2mm_M2, F.Cu at (52.5, 92.4)
- added REF**: MountingHole_2.2mm_M2, MountingHole:MountingHole_2.2mm_M2, F.Cu at (52.5, 69.1)
- added REF**: MountingHole_2.2mm_M2, MountingHole:MountingHole_2.2mm_M2, F.Cu at (75.8, 92.4)
- added REF**: MountingHole_2.2mm_M2, MountingHole:MountingHole_2.2mm_M2, F.Cu at (75.8, 69.1)
- added REF**: MountingHole_2.2mm_M2, MountingHole:MountingHole_2.2mm_M2, F.Cu at (338.0, 92.4)
- added REF**: MountingHole_2.2mm_M2, MountingHole:MountingHole_2.2mm_M2, F.Cu at (314.7, 92.4)
- added REF**: MountingHole_2.2mm_M2, MountingHole:MountingHole_2.2mm_M2, F.Cu at (314.7, 69.1)
- added REF**: MountingHole_2.2mm_M2, MountingHole:MountingHole_2.2mm_M2, F.Cu at (338.0, 69.1)
- moved J4 1.24 mm to (314.1, 39.1)
- moved J9 1.24 mm to (77.0, 33.8)
- moved U1 1.24 mm to (326.4, 50.5)
- moved U2 1.24 mm to (64.2, 50.5)
- moved J5 1.24 mm to (51.9, 39.1)
Routing:
- net ROT_A_R: track 100.9 -> 106.4 mm, vias 0 -> 2
- net ROW4_R: track 258.4 -> 263.6 mm
- net ROT_B_R: track 106.9 -> 111.8 mm, vias 0 -> 2
- net GND2: track 120.3 -> 124.9 mm
- net PERIPH_R: track 99.1 -> 102.7 mm
- net COL0: track 212.1 -> 215.0 mm
- net COL5: track 116.0 -> 118.0 mm
- net COL1_R: track 180.2 -> 181.7 mm
- net RESET_R: track 86.3 -> 87.8 mm
- net GND1: track 133.8 -> 132.3 mm
- net ROW0_R: track 149.4 -> 150.8 mm
- net ROW2: track 196.5 -> 198.0 mm
- net Net-(J9-Pad1): track 9.87 -> 11.1 mm
- net Net-(J4-Pad2): track 10.1 -> 11.3 mm
- net Net-(J9-Pad2): track 7.13 -> 8.37 mm
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Other:
- outline, holes or cut-outs redrawn

Commit message: Updated to V1.4.
Parts:
- removed J1, J6: OLED, Cantaloupe:OLED_0.96_SSD1306_128x64
- removed J3: ICSP, Connector_PinHeader_2.54mm:PinHeader_2x03_P2.54mm_Vertical
- removed J4: BAT_CON, Cantaloupe:Battery_Solder_Points
- removed J5: BAT_CON_R, Cantaloupe:Battery_Solder_Points
- removed J8: ICSP_R, Connector_PinHeader_2.54mm:PinHeader_2x03_P2.54mm_Vertical
- removed J9: BAT_CON_TOG, Cantaloupe:Battery_Solder_Points
- removed the REF** at (52.5, 92.4)
- removed the REF** at (52.5, 69.1)
- removed the REF** at (75.8, 92.4)
- removed the REF** at (75.8, 69.1)
- removed the REF** at (338.0, 92.4)
- removed the REF** at (314.7, 92.4)
- removed the REF** at (314.7, 69.1)
- removed the REF** at (338.0, 69.1)
- removed SW36: BAT_TOG, Cantaloupe:Switch_MSK-22D18
- removed SW72: BAT_TOG_R, Cantaloupe:Switch_MSK-22D18
- moved J2 24.1 mm to (337.8, 76.1)
- moved J7 24.1 mm to (52.7, 76.1)
- moved SW71 24.1 mm to (64.6, 76.2), turned to 90 degrees
- moved SW35 24.1 mm to (325.9, 76.2)
Connections:
- net PERIPH renamed COL6
- net PERIPH_R renamed COL6_R
- U1 pad 24: RAW -> Net-(U1-Pad24)
Routing:
- net COL3_R: track 219.7 -> 154.0 mm, vias 1 -> 0
- net COL4_R: track 168.2 -> 126.1 mm, vias 1 -> 0
- net RESET_R: track 87.8 -> 47.4 mm, vias 3 -> 0
- net RESET: track 85.9 -> 48.2 mm, vias 3 -> 1
- net ROW2: track 198.0 -> 163.6 mm
- net VCC: track 81.1 -> 47.9 mm
- net COL5_R: track 139.7 -> 107.5 mm
- net VDD: track 75.3 -> 43.8 mm
- net ROW3: track 214.9 -> 185.6 mm
- net SDA: track 26.9 -> 0.00 mm
- net SDA_R: track 26.2 -> 0.00 mm
- net SCL: track 26.1 -> 0.00 mm
- net SCL_R: track 25.4 -> 0.00 mm
- net DATA: track 65.3 -> 41.3 mm
- net DATA_R: track 70.4 -> 49.7 mm
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Other:
- board text added: "Cantaloupe V1.4 Aria"
- board text removed: "Cantaloupe V1.3 Aria"

Commit message: Added SMK support
Parts:
- removed G1: Art, Cantaloupe:Catmelon
- removed the G2 at (129.4, 119.8)
- added G2: Art, Cantaloupe:Catmelon, F.Cu at (64.9, 88.9)
- added G2: Art, Cantaloupe:Catmelon, F.Cu at (326.5, 88.9)
- SW1, SW10, SW11, SW12, SW13, SW14, SW15, SW16, SW17, SW18, SW19, SW2, SW20, SW21, SW22, SW23, SW24, SW25, SW26, SW27, SW28, SW29, SW3, SW30, SW34, SW37, SW38, SW39, SW4, SW40, SW41, SW42, SW43, SW44, SW45, SW46, SW47, SW48, SW49, SW5, SW50, SW51, SW52, SW53, SW54, SW55, SW56, SW57, SW58, SW59, SW6, SW60, SW61, SW62, SW63, SW64, SW65, SW66, SW7, SW70, SW8, SW9: footprint Cantaloupe:HYBRID-MX_ALPS-1U-NoLED -> Cantaloupe:HYBRID-MX_ALPS_SMK-1U-NoLED
- SW31, SW32, SW67, SW68: footprint Cantaloupe:HYBRID-MX_ALPS-2U-ReversedStabilizers-NoLED -> Cantaloupe:HYBRID-MX_ALPS_SMK-2U-ReversedStabilizers-NoLED
Routing:
- net COL2: track 162.0 -> 177.2 mm
- net COL1_R: track 181.7 -> 184.8 mm
- net COL3: track 152.4 -> 149.4 mm
- net COL0: track 215.0 -> 218.0 mm
- net ROW4_R: track 263.9 -> 266.8 mm
- net ROT_A: track 103.2 -> 106.0 mm
- net COL5_R: track 107.5 -> 105.0 mm
- net COL4_R: track 126.1 -> 128.5 mm
- net COL4: track 136.5 -> 134.6 mm
- net COL5: track 118.0 -> 119.9 mm
- net Net-(D25-Pad2): track 27.3 -> 28.5 mm
- net Net-(D56-Pad2): track 18.4 -> 19.3 mm
- net COL3_R: track 154.0 -> 154.9 mm
- net Net-(D61-Pad2): track 18.6 -> 19.2 mm

Commit message: Updated to V1.5.
Added the option for OLED again. Removed Alps support. Improved switch footprints. Removed 2u support and moved rotary encoder positions. Deleted 61st and 62nd keyswitches - now has exactly 30 switches per side. Changed USB C interconnect back to TRRS and moved position. Unified symbol libraries
Parts:
- removed G2 (x2): Art, Cantaloupe:Catmelon
- removed J7: Interconnect_R, Connector_USB:USB_C_Receptacle_HRO_TYPE-C-31-M-12
- removed the REF** at (193.7, 69.9)
- removed the REF** at (78.4, 121.5)
- removed the REF** at (174.6, 117.5)
- removed the REF** at (117.5, 112.7)
- removed the REF** at (98.4, 57.1)
- removed the REF** at (174.6, 60.3)
- removed the REF** at (196.8, 69.9)
- removed the REF** at (196.8, 108.0)
- removed the REF** at (193.7, 108.0)
- removed the REF** at (215.9, 60.3)
- removed the REF** at (215.9, 117.5)
- removed the REF** at (292.1, 57.1)
- removed the REF** at (273.1, 112.7)
- removed the REF** at (312.2, 121.5)
- removed SW65, SW66, SW70: MX, Cantaloupe:HYBRID-MX_ALPS_SMK-1U-NoLED
- removed SW67, SW68: MX, Cantaloupe:HYBRID-MX_ALPS_SMK-2U-ReversedStabilizers-NoLED
- removed SW69: Encoder_R, Rotary_Encoder:RotaryEncoder_Alps_EC11E-Switch_Vertical_H20mm
- removed SW71: Reset, Button_Switch_SMD:SW_SPST_TL3342
- added G***: LOGO, Cantaloupe:Catmelon, F.Cu at (222.1, 75.2)
- added G***: LOGO, Cantaloupe:Catmelon, F.Cu at (44.6, 76.9)
- added J1: MJ-4PP-9, Ariamelon:MJ-4PP-9_1side, F.Cu at (132.6, 152.5)
- added J3: MJ-4PP-9, Ariamelon:MJ-4PP-9_1side, F.Cu at (134.1, 152.5)
- added J4: OLED_R, Ariamelon:OLED_0.96_SSD1306_128x64, F.Cu at (194.6, 142.9)
- added REF**: MountingHole_4.3mm_M4, MountingHole:MountingHole_4.3mm_M4, F.Cu at (221.0, 125.4)
- added REF**: MountingHole_4.3mm_M4, MountingHole:MountingHole_4.3mm_M4, F.Cu at (215.1, 84.0)
- added REF**: MountingHole_4.3mm_M4, MountingHole:MountingHole_4.3mm_M4, F.Cu at (219.1, 31.7)
- added REF**: MountingHole_4.3mm_M4, MountingHole:MountingHole_4.3mm_M4, F.Cu at (161.9, 31.7)
- added REF**: MountingHole_4.3mm_M4, MountingHole:MountingHole_4.3mm_M4, F.Cu at (104.8, 31.7)
- added REF**: MountingHole_4.3mm_M4, MountingHole:MountingHole_4.3mm_M4, F.Cu at (47.6, 31.7)
- added REF**: MountingHole_2.2mm_M2, MountingHole:MountingHole_2.2mm_M2, F.Cu at (194.1, 154.7)
- added REF**: MountingHole_2.2mm_M2, MountingHole:MountingHole_2.2mm_M2, F.Cu at (194.1, 131.0)
- added REF**: MountingHole_2.2mm_M2, MountingHole:MountingHole_2.2mm_M2, F.Cu at (170.3, 131.0)
- added REF**: MountingHole_2.2mm_M2, MountingHole:MountingHole_2.2mm_M2, F.Cu at (170.3, 154.7)
- added REF**: MountingHole_2.2mm_M2, MountingHole:MountingHole_2.2mm_M2, F.Cu at (96.2, 154.7)
- added REF**: MountingHole_4.3mm_M4, MountingHole:MountingHole_4.3mm_M4, F.Cu at (51.6, 84.0)
- added REF**: MountingHole_2.2mm_M2, MountingHole:MountingHole_2.2mm_M2, F.Cu at (96.2, 131.0)
- added REF**: MountingHole_2.2mm_M2, MountingHole:MountingHole_2.2mm_M2, F.Cu at (72.4, 131.0)
- added REF**: MountingHole_2.2mm_M2, MountingHole:MountingHole_2.2mm_M2, F.Cu at (72.4, 154.7)
- added REF**: MountingHole_4.3mm_M4, MountingHole:MountingHole_4.3mm_M4, F.Cu at (158.7, 108.0)
- added REF**: MountingHole_4.3mm_M4, MountingHole:MountingHole_4.3mm_M4, F.Cu at (108.0, 108.0)
- added REF**: Breakaway_Tabs, Custom Parts:Breakaway_Tabs, F.Cu at (132.8, 74.2)
- added REF**: Breakaway_Tabs, Custom Parts:Breakaway_Tabs, F.Cu at (133.9, 74.2)
- added REF**: Breakaway_Tabs, Custom Parts:Breakaway_Tabs, F.Cu at (132.8, 151.6)
- added REF**: Breakaway_Tabs, Custom Parts:Breakaway_Tabs, F.Cu at (133.9, 151.6)
- added REF**: MountingHole_4.3mm_M4, MountingHole:MountingHole_4.3mm_M4, F.Cu at (45.7, 125.4)
- added SW36: MX, Ariamelon:HYBRID-MX_SMK-1U-NoLED, F.Cu at (147.6, 60.3)
- D1, D10, D11, D12, D13, D14, D15, D16, D17, D18, D19, D2, D20, D21, D22, D23, D24, D25, D26, D27, D28, D29, D3, D30, D31, D32, D33, D34, D35, D36, D37, D38, D39, D4, D40, D41, D42, D43, D44, D45, D46, D47, D48, D49, D5, D50, D51, D52, D53, D54, D55, D56, D57, D58, D59, D6, D60, D61, D62, D7, D8, D9: footprint Cantaloupe:D_Hybrid_SOD123_DO35 -> Ariamelon:D_Hybrid_SOD123_DO35
- J2: value Interconnect -> OLED_L; footprint Connector_USB:USB_C_Receptacle_HRO_TYPE-C-31-M-12 -> Ariamelon:OLED_0.96_SSD1306_128x64
- SW1, SW10, SW11, SW12, SW13, SW14, SW15, SW16, SW17, SW18, SW19, SW2, SW20, SW21, SW22, SW23, SW24, SW25, SW26, SW27, SW28, SW29, SW3, SW30, SW34, SW37, SW38, SW39, SW4, SW40, SW41, SW42, SW43, SW44, SW45, SW46, SW47, SW48, SW49, SW5, SW50, SW51, SW52, SW53, SW54, SW55, SW56, SW57, SW58, SW59, SW6, SW60, SW61, SW62, SW7, SW8, SW9: footprint Cantaloupe:HYBRID-MX_ALPS_SMK-1U-NoLED -> Ariamelon:HYBRID-MX_SMK-1U-NoLED
- SW31: value MX -> Encoder; footprint Cantaloupe:HYBRID-MX_ALPS_SMK-2U-ReversedStabilizers-NoLED -> Rotary_Encoder:RotaryEncoder_Alps_EC11E-Switch_Vertical_H20mm
- SW32: value MX -> Reset; footprint Cantaloupe:HYBRID-MX_ALPS_SMK-2U-ReversedStabilizers-NoLED -> Button_Switch_SMD:SW_SPST_TL3342
- SW33: value Encoder -> MX; footprint Rotary_Encoder:RotaryEncoder_Alps_EC11E-Switch_Vertical_H20mm -> Ariamelon:HYBRID-MX_SMK-1U-NoLED
- SW35: value Reset -> MX; footprint Button_Switch_SMD:SW_SPST_TL3342 -> Ariamelon:HYBRID-MX_SMK-1U-NoLED
- SW63: value MX -> Encoder; footprint Cantaloupe:HYBRID-MX_ALPS_SMK-1U-NoLED -> Rotary_Encoder:RotaryEncoder_Alps_EC11E-Switch_Vertical_H20mm
- SW64: value MX -> Reset; footprint Cantaloupe:HYBRID-MX_ALPS_SMK-1U-NoLED -> Button_Switch_SMD:SW_SPST_TL3342
- U1, U2: footprint Cantaloupe:ArduinoProMicro_Blank -> Ariamelon:ArduinoProMicro_Blank
- moved D30 306.5 mm to (22.8, 141.0), turned to 330 degrees
- moved SW30 290.7 mm to (26.8, 134.2), turned to 240 degrees
- moved J2 274.1 mm to (71.9, 142.9)
- moved D29 272.1 mm to (33.2, 121.6), turned to 345 degrees
- moved D31 266.3 mm to (49.7, 150.0), turned to 0 degrees
- moved SW29 262.7 mm to (35.2, 113.9), turned to 255 degrees
- moved SW32 257.4 mm to (64.9, 132.0), turned to 0 degrees
- moved D24 251.6 mm to (58.7, 125.4), turned to 0 degrees
- moved D28 247.4 mm to (38.2, 100.0), turned to 0 degrees
- moved SW24 243.1 mm to (58.7, 117.5), turned to 270 degrees
- moved SW28 240.7 mm to (38.1, 92.1), turned to 270 degrees
- moved D18 234.9 mm to (77.8, 125.4), turned to 0 degrees
- moved U1 229.9 mm to (114.6, 140.2), turned to 180 degrees
- moved D23 228.6 mm to (61.9, 106.4), turned to 0 degrees
- moved SW18 225.9 mm to (77.8, 117.5), turned to 270 degrees
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Connections:
- net COL1 renamed COL1_L
- net COL2 renamed COL2_L
- net COL3 renamed COL3_L
- net COL4 renamed COL4_L
- net COL5 renamed COL5_L
- net ROW0 renamed ROW0_L
- net ROW1 renamed ROW1_L
- net ROW2 renamed ROW2_L
- D19 pad 1: ROW3 -> ROW3_L
- D20 pad 1: ROW3 -> ROW3_L
- D21 pad 1: ROW3 -> ROW3_L
- D22 pad 1: ROW3 -> ROW3_L
- D23 pad 1: ROW3 -> ROW3_L
- D24 pad 1: ROW3 -> ROW3_L
- D25 pad 1: ROW4 -> ROW4_L
- D26 pad 1: ROW4 -> ROW4_L
- D27 pad 1: ROW4 -> ROW4_L
- D28 pad 1: ROW4 -> ROW4_L
- D29 pad 1: ROW4 -> ROW4_L
- D30 pad 1: ROW4 -> ROW4_L
- D31 pad 1: ROW4 -> ROW3_L
- D62 pad 1: ROW4_R -> ROW3_R
- SW1 pad 1: COL0 -> COL0_L
- SW13 pad 1: COL0 -> COL0_L
- SW19 pad 1: COL0 -> COL0_L
- SW25 pad 1: COL0 -> COL0_L
- SW32 pad 1: COL6 -> RESET_L
- SW32 pad 2: Net-(D31-Pad2) -> GND_L
- SW34 pad 1: Net-(D31-Pad2) -> Net-(D33-Pad2)
- SW34 pad 2: COL6 -> COL4_R
- SW35 pad 1: RESET -> Net-(D34-Pad2)
- SW35 pad 2: GND1 -> COL3_R
- SW37 pad 1: COL5_R -> Net-(D36-Pad2)
- SW37 pad 2: Net-(D32-Pad2) -> COL1_R
- SW38 pad 1: COL4_R -> Net-(D37-Pad2)
- SW38 pad 2: Net-(D33-Pad2) -> COL0_R
- SW39 pad 1: COL3_R -> Net-(D38-Pad2)
- SW39 pad 2: Net-(D34-Pad2) -> COL5_R
- SW40 pad 1: COL2_R -> Net-(D39-Pad2)
- SW40 pad 2: Net-(D35-Pad2) -> COL4_R
- SW41 pad 1: COL1_R -> Net-(D40-Pad2)
- SW41 pad 2: Net-(D36-Pad2) -> COL3_R
- SW42 pad 1: COL0_R -> Net-(D41-Pad2)
- SW42 pad 2: Net-(D37-Pad2) -> COL2_R
- SW43 pad 1: COL5_R -> Net-(D42-Pad2)
- SW43 pad 2: Net-(D38-Pad2) -> COL1_R
- SW44 pad 1: COL4_R -> Net-(D43-Pad2)
- SW44 pad 2: Net-(D39-Pad2) -> COL0_R
- SW45 pad 1: COL3_R -> Net-(D44-Pad2)
- SW45 pad 2: Net-(D40-Pad2) -> COL5_R
- SW46 pad 1: COL2_R -> Net-(D45-Pad2)
- SW46 pad 2: Net-(D41-Pad2) -> COL4_R
- SW47 pad 1: COL1_R -> Net-(D46-Pad2)
- SW47 pad 2: Net-(D42-Pad2) -> COL3_R
- SW48 pad 1: COL0_R -> Net-(D47-Pad2)
- SW48 pad 2: Net-(D43-Pad2) -> COL2_R
- SW49 pad 1: COL5_R -> Net-(D48-Pad2)
- SW49 pad 2: Net-(D44-Pad2) -> COL1_R
- SW50 pad 1: COL4_R -> Net-(D49-Pad2)
- SW50 pad 2: Net-(D45-Pad2) -> COL0_R
- SW51 pad 1: COL3_R -> Net-(D50-Pad2)
- SW51 pad 2: Net-(D46-Pad2) -> COL5_R
- SW52 pad 1: COL2_R -> Net-(D51-Pad2)
- SW52 pad 2: Net-(D47-Pad2) -> COL4_R
- SW53 pad 1: COL1_R -> Net-(D52-Pad2)
- SW53 pad 2: Net-(D48-Pad2) -> COL3_R
- SW54 pad 1: COL0_R -> Net-(D53-Pad2)
- SW54 pad 2: Net-(D49-Pad2) -> COL2_R
- SW55 pad 1: COL5_R -> Net-(D54-Pad2)
- SW55 pad 2: Net-(D50-Pad2) -> COL1_R
- SW56 pad 1: COL4_R -> Net-(D55-Pad2)
- SW56 pad 2: Net-(D51-Pad2) -> COL0_R
- SW57 pad 1: COL3_R -> Net-(D56-Pad2)
- SW57 pad 2: Net-(D52-Pad2) -> COL5_R
- SW58 pad 1: COL2_R -> Net-(D57-Pad2)
- SW58 pad 2: Net-(D53-Pad2) -> COL4_R
- SW59 pad 1: COL1_R -> Net-(D58-Pad2)
- SW59 pad 2: Net-(D54-Pad2) -> COL3_R
- SW60 pad 1: COL0_R -> Net-(D59-Pad2)
- SW60 pad 2: Net-(D55-Pad2) -> COL2_R
- SW61 pad 1: COL5_R -> Net-(D60-Pad2)
- SW61 pad 2: Net-(D56-Pad2) -> COL1_R
- SW62 pad 1: COL4_R -> Net-(D61-Pad2)
- SW62 pad 2: Net-(D57-Pad2) -> COL0_R
- SW64 pad 1: COL2_R -> RESET_R
- SW64 pad 2: Net-(D59-Pad2) -> GND_R
- SW7 pad 1: COL0 -> COL0_L
- U1 pad 1: ROT_B -> COL6_L
- U1 pad 10: ROW3 -> ROW3_L
- U1 pad 19: COL0 -> COL0_L
- U1 pad 2: DATA -> DATA_L
- U1 pad 21: VCC -> VDD_L
- U1 pad 22: RESET -> RESET_L
- U1 pad 23: GND1 -> Net-(U1-Pad23)
- U1 pad 4: Net-(U1-Pad4) -> GND_L
- U1 pad 5: SDA -> SDA_L
- U1 pad 6: SCL -> SCL_L
- U1 pad 7: ROT_A -> ROT_A_L
- U1 pad 8: COL6 -> ROT_B_L
- U1 pad 9: ROW4 -> ROW4_L
- U2 pad 10: COL3_R -> COL4_R
- U2 pad 11: COL4_R -> COL5_R
- U2 pad 12: COL5_R -> Net-(U2-Pad12)
- U2 pad 13: Net-(U2-Pad13) -> ROW1_R
- U2 pad 14: ROW1_R -> ROW2_R
- U2 pad 15: ROW2_R -> ROW3_R
- U2 pad 16: ROW3_R -> ROW4_R
- U2 pad 17: ROW4_R -> ROT_A_R
- U2 pad 18: COL6_R -> ROT_B_R
- U2 pad 19: ROT_B_R -> COL6_R
- U2 pad 2: DATA_R -> COL0_R
- U2 pad 20: ROT_A_R -> DATA_R
- U2 pad 21: VDD -> VDD_R
- U2 pad 23: GND2 -> GND_R
- U2 pad 7: COL0_R -> COL1_R
- U2 pad 8: COL1_R -> COL2_R
- U2 pad 9: COL2_R -> COL3_R
Routing:
- net ROW4: track 240.9 -> 0.00 mm
- net ROW4_L: track 0.00 -> 223.0 mm
- net COL0: track 218.0 -> 0.00 mm
- net COL0_L: track 0.00 -> 206.2 mm
- net ROW3_L: track 0.00 -> 199.3 mm
- net ROW3: track 185.6 -> 0.00 mm
- net GND2: track 142.1 -> 0.00 mm
- net GND1: track 140.6 -> 0.00 mm, vias 1 -> 0
- net COL6: track 120.9 -> 0.00 mm
- net GND_L: track 0.00 -> 117.0 mm
- net ROT_B: track 112.8 -> 0.00 mm
- net ROT_A: track 106.0 -> 0.00 mm
- net VDD_L: track 0.00 -> 104.1 mm
- net COL6_L: track 0.00 -> 98.0 mm
- net ROT_B_L: track 0.00 -> 98.0 mm
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Other:
- board size 289.7 x 117 mm -> 238.4 x 143.9 mm
- board text added: "Cantaloupe V1.5 Aria"
- board text added: "OLED"
- board text removed: "Cantaloupe V1.4 Aria"

Commit message: New ARM variant (experimental WIP)
Parts:
- removed D33, D34, D35, D36, D37, D38, D39, D40, D41, D42, D43, D44, D45, D46, D47, D48, D49, D50, D51, D52, D53, D54, D55, D56, D57, D58, D59, D60, D61, D62: D, Ariamelon:D_Hybrid_SOD123_DO35
- removed G*** (x2): LOGO, Cantaloupe:Catmelon
- removed REF** (x10): MountingHole_4.3mm_M4, MountingHole:MountingHole_4.3mm_M4
- removed REF** (x8): MountingHole_2.2mm_M2, MountingHole:MountingHole_2.2mm_M2
- removed REF** (x4): Breakaway_Tabs, Custom Parts:Breakaway_Tabs
- removed SW33, SW34, SW35, SW36, SW37, SW38, SW39, SW40, SW41, SW42, SW43, SW44, SW45, SW46, SW47, SW48, SW49, SW50, SW51, SW52, SW53, SW54, SW55, SW56, SW57, SW58, SW59, SW60, SW61, SW62: MX, Ariamelon:HYBRID-MX_SMK-1U-NoLED
- removed SW63: Encoder, Rotary_Encoder:RotaryEncoder_Alps_EC11E-Switch_Vertical_H20mm
- removed SW64: Reset, Button_Switch_SMD:SW_SPST_TL3342
- added A1: Art, Ariamelon:Catmelon, F.Cu at (144.3, 53.4)
- added C1: 100n, Capacitor_SMD:C_0603_1608Metric, B.Cu at (152.4, 80.8)
- added C10: 20p, Capacitor_SMD:C_0603_1608Metric, B.Cu at (144.4, 62.6)
- added C11: 100n, Capacitor_SMD:C_0603_1608Metric, B.Cu at (136.7, 61.3)
- added C12: 20p, Capacitor_SMD:C_0603_1608Metric, B.Cu at (139.6, 65.4)
- added C13: 100n, Capacitor_SMD:C_0603_1608Metric, B.Cu at (135.5, 50.7)
- added C14: 100n, Capacitor_SMD:C_0603_1608Metric, B.Cu at (149.9, 61.5)
- added C2: 10u, Capacitor_SMD:C_0603_1608Metric, B.Cu at (150.4, 52.0)
- added C3: 100n, Capacitor_SMD:C_0603_1608Metric, B.Cu at (133.6, 80.8)
- added C4: 1u, Capacitor_SMD:C_0603_1608Metric, B.Cu at (155.1, 53.8)
- added C5: 10u, Capacitor_SMD:C_0603_1608Metric, B.Cu at (140.0, 108.2)
- added C6: 10u, Capacitor_SMD:C_0603_1608Metric, B.Cu at (136.6, 37.2)
- added C7: 10u, Capacitor_SMD:C_0603_1608Metric, B.Cu at (137.3, 42.8)
- added C8: 100n, Capacitor_SMD:C_0603_1608Metric, B.Cu at (147.1, 50.2)
- added C9: 100n, Capacitor_SMD:C_0603_1608Metric, B.Cu at (149.9, 59.8)
- added F1: 1A, Fuse:Fuse_1206_3216Metric, B.Cu at (144.4, 102.1)
- added F2: 2A, Fuse:Fuse_1206_3216Metric, B.Cu at (139.2, 25.8)
- added H1: M2, Ariamelon:MountingHole_2.2mm_M2_Pad, F.Cu at (32.4, 43.8)
- added H2: M2, Ariamelon:MountingHole_2.2mm_M2_Pad, F.Cu at (32.4, 101.0)
- added H3: M2, Ariamelon:MountingHole_2.2mm_M2_Pad, F.Cu at (70.5, 36.0)
- added H4: M2, Ariamelon:MountingHole_2.2mm_M2_Pad, F.Cu at (70.5, 93.1)
- added H5: M2, Ariamelon:MountingHole_2.2mm_M2_Pad, F.Cu at (108.5, 39.6)
- added H6: M2, Ariamelon:MountingHole_2.2mm_M2_Pad, F.Cu at (108.6, 96.7)
- added H7: M2, Ariamelon:MountingHole_2.2mm_M2_Pad, F.Cu at (153.8, 18.1)
- added H8: M2, Ariamelon:MountingHole_2.2mm_M2_Pad, F.Cu at (152.2, 99.9)
- added J5: Trackball, Ariamelon:pimoroni_trackball_flippable, F.Cu at (143.0, 89.8)
- added JP1: Side_L, Jumper:SolderJumper-2_P1.3mm_Open_Pad1.0x1.5mm, F.Cu at (149.5, 71.4)
- added JP2: Side_R, Jumper:SolderJumper-2_P1.3mm_Open_Pad1.0x1.5mm, B.Cu at (149.5, 71.4)
- added JP3: Link-_L, Jumper:SolderJumper-2_P1.3mm_Open_Pad1.0x1.5mm, F.Cu at (138.5, 102.7)
- added JP4: Link+_L, Jumper:SolderJumper-2_P1.3mm_Open_Pad1.0x1.5mm, F.Cu at (137.3, 104.9)
- added JP5: Link-_R, Jumper:SolderJumper-2_P1.3mm_Open_Pad1.0x1.5mm, B.Cu at (138.5, 102.7)
- added JP6: Link+_R, Jumper:SolderJumper-2_P1.3mm_Open_Pad1.0x1.5mm, B.Cu at (137.3, 104.9)
- added Q1: 2N7002, Package_TO_SOT_SMD:SOT-23, B.Cu at (155.1, 56.5)
- added Q2: AO3401A, Package_TO_SOT_SMD:SOT-23, B.Cu at (137.4, 30.3)
- added R1: 10k, Resistor_SMD:R_0603_1608Metric, B.Cu at (152.4, 77.5)
- added R10: 10k, Resistor_SMD:R_0603_1608Metric, B.Cu at (133.6, 79.0)
- added R11: 10k, Resistor_SMD:R_0603_1608Metric, B.Cu at (155.1, 59.3)
- added R12: 10k, Resistor_SMD:R_0603_1608Metric, B.Cu at (133.6, 77.2)
- added R13: 100k, Resistor_SMD:R_0603_1608Metric, B.Cu at (136.1, 27.3)
- added R14: 200k, Resistor_SMD:R_0603_1608Metric, B.Cu at (136.1, 24.3)
- added R15: 2k2, Resistor_SMD:R_0603_1608Metric, B.Cu at (133.7, 35.1)
- added R16: 10k, Resistor_SMD:R_0603_1608Metric, B.Cu at (149.5, 68.1)
- added R17: 220, Resistor_SMD:R_0603_1608Metric, B.Cu at (141.1, 62.6)
- added R2: 33, Resistor_SMD:R_0603_1608Metric, B.Cu at (142.4, 47.8)
- added R3: 33, Resistor_SMD:R_0603_1608Metric, B.Cu at (144.1, 47.8)
- added R4: 1k5, Resistor_SMD:R_0603_1608Metric, B.Cu at (145.9, 47.8)
- added R5: 5k1, Resistor_SMD:R_0603_1608Metric, B.Cu at (136.4, 21.0)
- added R6: 5k1, Resistor_SMD:R_0603_1608Metric, B.Cu at (149.1, 23.9)
- added R7: 10k, Resistor_SMD:R_0603_1608Metric, B.Cu at (150.4, 50.2)
- added R8: 10k, Resistor_SMD:R_0603_1608Metric, B.Cu at (152.4, 79.1)
- added R9: 100k, Resistor_SMD:R_0603_1608Metric, B.Cu at (150.4, 53.8)
- added U3: SRV05-4, Package_TO_SOT_SMD:SOT-23-6, B.Cu at (141.2, 105.7)
- added U4: XC6206P332MR, Package_TO_SOT_SMD:SOT-23, B.Cu at (137.3, 40.0)
- added U5: LMV321, Package_TO_SOT_SMD:SOT-23-5, B.Cu at (137.3, 34.4)
- added Y1: 8MHz, Crystal:Crystal_SMD_3225-4Pin_3.2x2.5mm, B.Cu at (142.6, 65.4)
- D1, D10, D11, D12, D13, D14, D15, D16, D17, D18, D19, D2, D20, D21, D22, D23, D24, D25, D26, D27, D28, D29, D3, D30, D31, D4, D5, D6, D7, D8, D9: footprint Ariamelon:D_Hybrid_SOD123_DO35 -> Ariamelon:D_SOD-123
- D32: value D -> Power; footprint Ariamelon:D_Hybrid_SOD123_DO35 -> Ariamelon:LED_0603_1608Metric_Flippable; moved to F.Cu
- J1: value MJ-4PP-9 -> USB_In; footprint Ariamelon:MJ-4PP-9_1side -> Ariamelon:USB-C-C168688; moved to B.Cu
- J2: value OLED_L -> OLED; footprint Ariamelon:OLED_0.96_SSD1306_128x64 -> Ariamelon:OLED_0.96_SSD1306_128x64_Flippable
- J3: value MJ-4PP-9 -> Link; footprint Ariamelon:MJ-4PP-9_1side -> Ariamelon:USB-C-C168688; moved to B.Cu
- J4: value OLED_R -> Debug; footprint Ariamelon:OLED_0.96_SSD1306_128x64 -> Ariamelon:Debug_JTAG_SWD
- SW1, SW10, SW11, SW12, SW13, SW14, SW15, SW16, SW17, SW18, SW19, SW2, SW20, SW21, SW22, SW23, SW24, SW25, SW26, SW27, SW28, SW29, SW3, SW30, SW4, SW5, SW6, SW7, SW8, SW9: footprint Ariamelon:HYBRID-MX_SMK-1U-NoLED -> Ariamelon:MXOnly-1U-Hotswap-Dual
- SW31: footprint Rotary_Encoder:RotaryEncoder_Alps_EC11E-Switch_Vertical_H20mm -> Ariamelon:EC11_Flippable
- SW32: value Reset -> MX; footprint Button_Switch_SMD:SW_SPST_TL3342 -> Ariamelon:Switch_TS24CA_Flippable; moved to B.Cu
- U1: value ProMicro -> STM32F303CCTx; footprint Ariamelon:ArduinoProMicro_Blank -> Package_QFP:LQFP-48_7x7mm_P0.5mm
- U2: value ProMicro -> SRV05-4; footprint Ariamelon:ArduinoProMicro_Blank -> Package_TO_SOT_SMD:SOT-23-6
- moved SW32 141.2 mm to (156.3, 24.4), turned to 90 degrees
- moved J1 138.0 mm to (143.5, 15.0), turned to 180 degrees
- moved J4 119.1 mm to (141.6, 36.2), turned to 0 degrees
- moved U2 114.4 mm to (143.3, 26.1), turned to 270 degrees
- moved SW30 108.8 mm to (134.8, 120.7), turned to 330 degrees
- moved SW31 107.0 mm to (143.0, 89.8), turned to 270 degrees
- moved D30 106.7 mm to (126.5, 115.9), turned to 60 degrees
- moved D31 104.6 mm to (141.4, 99.7)
- moved J2 101.1 mm to (143.0, 71.0), turned to 180 degrees
- moved D6 94.6 mm to (127.6, 31.6), turned to 90 degrees
- moved SW1 92.4 mm to (22.9, 35.6), turned to 0 degrees
- moved D29 90.8 mm to (123.8, 114.7), turned to 75 degrees
- moved SW25 90.8 mm to (22.9, 111.8), turned to 0 degrees
- moved U1 89.0 mm to (142.2, 55.5), turned to 90 degrees
- moved D32 88.6 mm to (133.7, 38.5), turned to 270 degrees
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Connections:
- D1 pad 1: ROW0_L -> ROW0
- D10 pad 1: ROW1_L -> ROW1
- D11 pad 1: ROW1_L -> ROW1
- D12 pad 1: ROW1_L -> ROW1
- D13 pad 1: ROW2_L -> ROW2
- D14 pad 1: ROW2_L -> ROW2
- D15 pad 1: ROW2_L -> ROW2
- D16 pad 1: ROW2_L -> ROW2
- D17 pad 1: ROW2_L -> ROW2
- D18 pad 1: ROW2_L -> ROW2
- D19 pad 1: ROW3_L -> ROW3
- D2 pad 1: ROW0_L -> ROW0
- D20 pad 1: ROW3_L -> ROW3
- D21 pad 1: ROW3_L -> ROW3
- D22 pad 1: ROW3_L -> ROW3
- D23 pad 1: ROW3_L -> ROW3
- D24 pad 1: ROW3_L -> ROW3
- D25 pad 1: ROW4_L -> ROW4
- D26 pad 1: ROW4_L -> ROW4
- D27 pad 1: ROW4_L -> ROW4
- D28 pad 1: ROW4_L -> ROW4
- D29 pad 1: ROW4_L -> ROW4
- D3 pad 1: ROW0_L -> ROW0
- D30 pad 1: ROW4_L -> ROW4
- D31 pad 1: ROW3_L -> ROW3
- D32 pad 1: ROW0_R -> Net-(D32-Pad1)
- D32 pad 2: Net-(D32-Pad2) -> VDD
- D4 pad 1: ROW0_L -> ROW0
- D5 pad 1: ROW0_L -> ROW0
- D6 pad 1: ROW0_L -> ROW0
- D7 pad 1: ROW1_L -> ROW1
- D8 pad 1: ROW1_L -> ROW1
- D9 pad 1: ROW1_L -> ROW1
- J2 pad 1: GND_L -> GND
- J2 pad 2: VDD_L -> VDD
- J2 pad 3: SCL_L -> SCL
- J2 pad 4: SDA_L -> SDA
- J4 pad 1: GND_R -> GND
- J4 pad 2: VDD_R -> JTDI
- J4 pad 3: SCL_R -> JTD0
- J4 pad 4: SDA_R -> JTCK
- SW1 pad 1: COL0_L -> COL0
- SW10 pad 1: COL3_L -> COL3
- SW11 pad 1: COL4_L -> COL4
- SW12 pad 1: COL5_L -> COL5
- SW13 pad 1: COL0_L -> COL0
- SW14 pad 1: COL1_L -> COL1
- SW15 pad 1: COL2_L -> COL2
- SW16 pad 1: COL3_L -> COL3
- SW17 pad 1: COL4_L -> COL4
- SW18 pad 1: COL5_L -> COL5
- SW19 pad 1: COL0_L -> COL0
- SW2 pad 1: COL1_L -> COL1
- SW20 pad 1: COL1_L -> COL1
- SW21 pad 1: COL2_L -> COL2
- SW22 pad 1: COL3_L -> COL3
- SW23 pad 1: COL4_L -> COL4
- SW24 pad 1: COL5_L -> COL5
- SW25 pad 1: COL0_L -> COL0
- SW26 pad 1: COL1_L -> COL1
- SW27 pad 1: COL2_L -> COL2
- SW28 pad 1: COL3_L -> COL3
- SW29 pad 1: COL4_L -> COL4
- SW3 pad 1: COL2_L -> COL2
- SW30 pad 1: COL5_L -> Net-(D30-Pad2)
- SW30 pad 2: Net-(D30-Pad2) -> COL5
- SW31 pad A: ROT_A_L -> Net-(C1-Pad2)
- SW31 pad B: ROT_B_L -> Net-(C3-Pad2)
- SW31 pad C: GND_L -> GND
- SW31 pad S1: Net-(D31-Pad2) -> COLROT
- SW31 pad S2: COL6_L -> Net-(D31-Pad2)
- SW32 pad 1: RESET_L -> BOOT0
- SW32 pad 2: GND_L -> VDD
- SW4 pad 1: COL3_L -> COL3
- SW5 pad 1: COL4_L -> COL4
- SW6 pad 1: COL5_L -> COL5
- SW7 pad 1: COL0_L -> COL0
- SW8 pad 1: COL1_L -> COL1
- SW9 pad 1: COL2_L -> COL2
- U1 pad 1: COL6_L -> VDD
- U1 pad 10: ROW3_L -> Net-(U1-Pad10)
- U1 pad 11: ROW2_L -> Net-(U1-Pad11)
- U1 pad 12: ROW1_L -> Net-(U1-Pad12)
- U1 pad 14: COL5_L -> ROT_B
- U1 pad 15: COL4_L -> COLROT
- U1 pad 16: COL3_L -> ROW4
- U1 pad 17: COL2_L -> ROW3
- U1 pad 18: COL1_L -> ROW2
- U1 pad 19: COL0_L -> COL5
- U1 pad 2: DATA_L -> Side
- U1 pad 20: ROW0_L -> COL4
- U1 pad 21: VDD_L -> TX
- U1 pad 22: RESET_L -> RX
- U1 pad 23: Net-(U1-Pad23) -> GND
- U1 pad 24: Net-(U1-Pad24) -> VDD
- U1 pad 4: GND_L -> Net-(U1-Pad4)
- U1 pad 5: SDA_L -> HSE_IN
- U1 pad 6: SCL_L -> HSE_OUT
- U1 pad 7: ROT_A_L -> NRST
- U1 pad 8: ROT_B_L -> GND
- U1 pad 9: ROW4_L -> VDD
- U2 pad 1: ROW0_R -> D-
- U2 pad 2: COL0_R -> GND
- U2 pad 3: Net-(U2-Pad3) -> D+
- U2 pad 5: SDA_R -> VBUS
- U2 pad 6: SCL_R -> Net-(U2-Pad6)
Routing:
- net ROW4_L: track 223.0 -> 0.00 mm
- net ROW4_R: track 218.7 -> 0.00 mm
- net COL0: track 0.00 -> 216.9 mm
- net COL0_R: track 213.5 -> 0.00 mm
- net COL0_L: track 206.2 -> 0.00 mm
- net ROW3_L: track 199.3 -> 0.00 mm
- net ROW3_R: track 197.2 -> 0.00 mm
- net COL1: track 0.00 -> 194.4 mm
- net COL1_L: track 185.3 -> 0.00 mm
- net COL1_R: track 182.2 -> 0.00 mm
- net VDD: track 0.00 -> 181.2 mm, vias 0 -> 12
- net COL2: track 0.00 -> 171.9 mm
- net ROW4: track 0.00 -> 168.7 mm
- net ROW3: track 0.00 -> 166.7 mm, vias 0 -> 2
- net COL3: track 0.00 -> 162.8 mm
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- added copper zone on B.Cu, net GND
- added copper zone on F.Cu, net GND
Other:
- board size 238.4 x 143.9 mm -> 143.9 x 118.7 mm
- net class Battery: clearance 0.2 -> 0.127
- net class Default: clearance 0.2 -> 0.127; trace_width 0.25 -> 0.2; via_dia 0.7 -> 0.45; via_drill 0.35 -> 0.3
- net class Power: clearance 0.2 -> 0.127; via_dia 0.7 -> 0.6; via_drill 0.35 -> 0.3
- rule trace_clearance: 0.2 -> 0.127
- board text added: "Cantaloupe V2.0 Aria"
- board text added: "Encoder"
- board text added: "Trackball"
- board text removed: "Cantaloupe V1.5 Aria"
