File: V2/PCB/Cantaloupe.sch (KiCad schematic (older format))
At the start: 120 parts, among them J1 USB_In, J2 OLED, J3 Link, J4 Debug, J5 Trackball, Q1 2N7002, Q2 AO3401A, SW1 MX, SW10 MX, SW11 MX, SW12 MX, SW13 MX, SW14 MX, SW15 MX, SW16 MX, SW17 MX, SW18 MX, SW19 MX, SW2 MX, SW20 MX, SW21 MX, SW22 MX, SW23 MX, SW24 MX, SW25 MX, SW26 MX, SW27 MX, SW28 MX, SW29 MX, SW3 MX, SW30 MX, SW31 Encoder, SW32 MX, SW4 MX, SW5 MX, SW6 MX, SW7 MX, SW8 MX, SW9 MX, U1 STM32F4x1CxUx, U2 SRV05-4, U3 SRV05-4, U4 XC6206P332MR, U5 LMV321, Y1 8MHz

Commit message: Fixed many issues with the board
Changed pin assignments so B2 isn't used. Added pull-up for RX pin and pull-down for B2 pin so the keyboard can properly load into the bootloader. Changed reset circuit so it actually works. Removed USB series resistors. Removed non-functional JTAG pins. Changed SRV05-04 to SRV0504. Thanks to sigprof and MasterSpoon from the QMK discord server for the help!
Parts:
- added D33: D, Ariamelon:D_SOD-123, symbol Device:D_Small
- C4: value 1u -> 100n
- J4: symbol Connector_Generic:Conn_01x06 -> Connector_Generic:Conn_01x04
- R11: value 10k -> 1M
- R2: value 10 -> 330k
- R3: value 10 -> 1k
- R9: value 100k -> 100
- U2, U3: value SRV05-4 -> SRV0504
Connections:
- net BOOT0: now also C2.1, R11.1, R2.1; no longer C2.2, R7.2, SW32.1 (A)
- net D+: now also U1.33 (PA12); no longer R3.1
- net D-: now also U1.32 (PA11); no longer R2.1
- net GND: now also C2.2, J4.4 (Pin_4), R11.2; no longer J4.6 (Pin_6), R9.2
- net NRST: now also R9.2; no longer Q1.3 (D), R11.2
- net VBUS: no longer U2.5 (VP)
- net VDD: no longer R11.1
- net at R2.2: now also D33.1 (K); no longer U1.32 (PA11)
- net at R3.2: now also Q1.1 (G), R7.2; no longer U1.33 (PA12)
- net V_ESD: now reaches F2.1, Q2.3 (D), R13.1, U5.3 (-)
- net V_ESD: now also U2.5 (VP)
- net JTCK renamed SWOCLK
- net JTD0: no longer names the net of U1.39 (PB3)
- net JTD0: no longer J4.4 (Pin_4)
- net JTDI: no longer names the net of U1.38 (PA15)
- net JTDI: no longer J4.5 (Pin_5)
- net JTMS renamed SWOIO
- new net: D33.2 (A), R3.1, SW32.1 (A)
- new net: Q1.3 (D), R9.1
- no-connect marks 18 -> 20
Other:
- moved on the sheet: A1, C10, C12, C2, C4, F1, F2, JP1, JP2, Q1, Q2, R13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
