File: PCB/Cantaloupe.kicad_pcb (KiCad board)
At the start: 2 copper layers, 155.5 x 134.4 mm, 204 parts, among them J1 SWD, J2 TC2030-NL, J3 VIK Keyboard Expansion, J4 OLED Breakout, J5 RGB_EX, J6 USB In, Q1 BSS138BKS, Q2 AO3401A, SW1 CPG151101S11, SW10 CPG151101S11, SW11 CPG151101S11, SW12 CPG151101S11, SW13 CPG151101S11, SW14 CPG151101S11, SW15 CPG151101S11, SW16 CPG151101S11, SW17 CPG151101S11, SW18 CPG151101S11, SW19 CPG151101S11, SW2 CPG151101S11, SW20 CPG151101S11, SW21 CPG151101S11, SW22 CPG151101S11, SW23 CPG151101S11, SW24 CPG151101S11, SW25 CPG151101S11, SW26 CPG151101S11, SW27 CPG151101S11, SW28 CPG151101S11, SW29 CPG151101S11, SW3 CPG151101S11, SW30 CPG151101S11, SW31 CPG151101S11, SW4 CPG151101S11, SW5 CPG151101S11, SW6 CPG151101S11, SW67 PTS645, SW68 PTS645, SW7 CPG151101S11, SW8 CPG151101S11, SW9 CPG151101S11, U1 ZD25WQ32CEIGR, U10 XC6206P332MR, U12 TPD4E05U06, U2 RP2040, U3 SN74AHCT1G125, U4 REF3033, U5 TUSB321, U6 74HC595, U8 INA180A4, U9 TPS259533, Y1 12MHz

Commit message: 23/08/2023 update
Changed MCU to nRF52840. Added nPM1300 PMIC for power management. Replaced SSD1351 display with Nice!View. Added Kailh Choc V1/V2 and Gateron KS-27/KS-33 support.
Parts:
- removed A2: VIK Logo, Cantaloupe:vik-logo-medium
- removed C1, C2: 100n, Capacitor_SMD:C_0402_1005Metric
- removed C34: 47u, Capacitor_SMD:C_1206_3216Metric
- removed C35, C36: 1u, Capacitor_SMD:C_0402_1005Metric
- removed C37, C38, C39, C40, C41, C42, C43, C44, C45, C46, C47, C48, C49, C50, C51, C52, C53, C54, C55, C56, C57, C58, C59, C60, C61, C62, C63: 100n, Cantaloupe:C_0402_1005Metric
- removed the D1 at (82.4, 53.0)
- removed the D10 at (139.5, 61.0)
- removed the D11 at (158.6, 64.9)
- removed the D12 at (177.6, 68.1)
- removed the D13 at (82.4, 91.1)
- removed the D14 at (101.4, 88.8)
- removed the D15 at (120.5, 84.0)
- removed D18, D19, D20, D21, D22, D23, D24, D25, D26, D27, D28, D29, D30, D47: SK6812MINI-E, Cantaloupe:YS-SK6812MINI-E
- removed the D2 at (101.4, 50.7)
- removed the D3 at (120.5, 45.9)
- removed the D4 at (139.5, 41.9)
- removed D46: BAV70, Cantaloupe:SOT-23-3
- removed the D5 at (158.6, 45.9)
- removed the D6 at (177.6, 49.1)
- removed D65: 1N4148, Cantaloupe:D_SOD-323
- removed the D7 at (82.4, 72.1)
- removed the D8 at (101.4, 69.7)
- removed the D9 at (120.5, 64.9)
- removed D98: 5V, Diode_SMD:D_SOD-523
- removed H10, H11, H8, H9: M3, Cantaloupe:MountingHole_3.2mm_M3_Pad
- removed H14, H15, H16, H17: M2, MountingHole:MountingHole_2.2mm_M2_Pad
- removed JP1: RGB_OUT_SEL, Jumper:SolderJumper-3_P1.3mm_Open_Pad1.0x1.5mm_NumberLabels
- removed Q2: AO3401A, Cantaloupe:SOT-23-3
- removed R12: 0.005, Resistor_SMD:R_0805_2012Metric
- removed R13, R15, R16, R18, R23, R24: 10k, Resistor_SMD:R_0402_1005Metric
- removed R14: 15k, Resistor_SMD:R_0402_1005Metric
- removed R17: 12k, Resistor_SMD:R_0402_1005Metric
- removed R19: 6k8, Resistor_SMD:R_0402_1005Metric
- removed R20, R22: 2k, Resistor_SMD:R_0402_1005Metric
- removed R21: 4k7, Resistor_SMD:R_0402_1005Metric
- removed REF**: HRS_CX70M-24P1, Cantaloupe:HRS_CX70M-24P1
- removed SW67, SW68: PTS645, Cantaloupe:SW_SPST_PTS645
- removed U10: XC6206P332MR, Cantaloupe:SOT-23-3
- removed U12: TPD4E05U06, Cantaloupe:USON-10_2.5x1.0mm_P0.5mm
- removed U8: INA180A4, Package_TO_SOT_SMD:SOT-23-5
- removed U9: TPS259533, Cantaloupe:WSON-8-1EP_2x2mm_P0.5mm_EP0.9x1.6mm
- added L1: 2u2, Cantaloupe:L_Murata_DFE201610P, B.Cu at (201.3, 47.9)
- added L2: 470n, Cantaloupe:L_Murata_DFE201610P, B.Cu at (199.9, 80.3)
- added L3: 10u, Cantaloupe:L_0603_1608Metric, B.Cu at (196.2, 56.4)
- added L4: 15n, Cantaloupe:L_0402_1005Metric, B.Cu at (195.9, 55.4)
- added L5: 4n7, Cantaloupe:L_0402_1005Metric, B.Cu at (256.8, 87.7)
- added L6: 2n2, Cantaloupe:L_0402_1005Metric, B.Cu at (258.8, 88.2)
- added R10: 732k, Cantaloupe:R_0402_1005Metric, B.Cu at (199.5, 76.4)
- added R11: 100k, Cantaloupe:R_0402_1005Metric, B.Cu at (201.2, 76.4)
- added R8: 10k, Cantaloupe:R_0402_1005Metric, B.Cu at (137.3, 131.0)
- added R9: 100k, Cantaloupe:R_0402_1005Metric, B.Cu at (201.6, 77.6)
- added SW32: RotaryEncoder, Cantaloupe:EVQVVD00203B-Flippable, B.Cu at (134.0, 145.8)
- added SW33: Bat_SW, Button_Switch_SMD:SW_SPDT_PCM12, B.Cu at (186.5, 39.2)
- added Y2: 32.768k, Crystal:Crystal_SMD_2012-2Pin_2.0x1.2mm, B.Cu at (200.0, 58.9)
- A1: footprint Cantaloupe:Ariamelon_Logo_x3_Mask -> Cantaloupe:Ariamelon_Logo_x2_CU
- C10, C28, C8: value 100n -> 1u; footprint Capacitor_SMD:C_0402_1005Metric -> Cantaloupe:C_0402_1005Metric
- C11, C12, C13, C16: value 100n -> 10u; footprint Capacitor_SMD:C_0402_1005Metric -> Cantaloupe:C_0603_1608Metric
- C14, C6: value 100n -> 10n; footprint Capacitor_SMD:C_0402_1005Metric -> Cantaloupe:C_0402_1005Metric
- C15: value 30p -> 10n; footprint Capacitor_SMD:C_0402_1005Metric -> Cantaloupe:C_0402_1005Metric
- C17: value 30p -> 22u; footprint Capacitor_SMD:C_0402_1005Metric -> Cantaloupe:C_0805_2012Metric
- C18: value 470n -> 100n; footprint Capacitor_SMD:C_0603_1608Metric -> Cantaloupe:C_0402_1005Metric
- C19: value 10n -> 22p; footprint Capacitor_SMD:C_0402_1005Metric -> Cantaloupe:C_0402_1005Metric
- C20, C3: value 1u -> 22p; footprint Capacitor_SMD:C_0402_1005Metric -> Cantaloupe:C_0402_1005Metric
- C21, C26: value 100n -> 4u7; footprint Capacitor_SMD:C_0402_1005Metric -> Cantaloupe:C_0402_1005Metric
- C22: value 10n -> 100n; footprint Capacitor_SMD:C_0402_1005Metric -> Cantaloupe:C_0402_1005Metric
- C23: value 1u -> 100p; footprint Capacitor_SMD:C_0603_1608Metric -> Cantaloupe:C_0402_1005Metric
- C24: value 100n -> 1p
- C25: value 100n -> 1p2
- C27: value 100n -> 4u7
- C29, C30, C9: footprint Capacitor_SMD:C_0402_1005Metric -> Cantaloupe:C_0402_1005Metric
- C31, C5: value 1u -> 100n; footprint Capacitor_SMD:C_0402_1005Metric -> Cantaloupe:C_0402_1005Metric
- C32: value 47u -> 1u; footprint Capacitor_SMD:C_1206_3216Metric -> Cantaloupe:C_0402_1005Metric
- C33: value 47u -> 100n; footprint Capacitor_SMD:C_1206_3216Metric -> Cantaloupe:C_0402_1005Metric
- C4: value 4u7 -> 22p; footprint Capacitor_SMD:C_0603_1608Metric -> Cantaloupe:C_0402_1005Metric
- C7: value 100n -> 1u; footprint Capacitor_SMD:C_0402_1005Metric -> Cantaloupe:C_0603_1608Metric
- D16: value SK6812MINI-E -> 5V; footprint Cantaloupe:YS-SK6812MINI-E -> Diode_SMD:D_SOD-523
- D17: value SK6812MINI-E -> S310F3WT; footprint Cantaloupe:YS-SK6812MINI-E -> Cantaloupe:LED_Lite-On_LTST-S310_3x1.5mm_Horizontal
- FB1: value 50R@100MHz -> 60R; footprint Inductor_SMD:L_1206_3216Metric -> Cantaloupe:L_0805_2012Metric
- H7: moved to F.Cu
- J1: value SWD -> TC2030-NL; footprint Cantaloupe:Header_SWD -> Connector:Tag-Connect_TC2030-IDC-NL_2x03_P1.27mm_Vertical
- J2: value TC2030-NL -> Nice!View; footprint Connector:Tag-Connect_TC2030-IDC-NL_2x03_P1.27mm_Vertical -> Cantaloupe:Nice!View_Flippable
- J3: value VIK Keyboard Expansion -> USB_C_Receptacle; footprint Cantaloupe:vik-keyboard-connector-horizontal -> Cantaloupe:HRS_CX70M-24P1
- J4: value OLED Breakout -> Bat; footprint Cantaloupe:OLED_1.5_SSD1351_128x128 -> Cantaloupe:JST_SH_SM03B-SRSS-TB_1x03-1MP_P1.00mm_Horizontal; moved to B.Cu
- J5: value RGB_EX -> VIK Keyboard; footprint Cantaloupe:Header_RGB -> Cantaloupe:VIK-Keyboard-Connector-Horizontal
- J6: value USB In -> U.FL; footprint Cantaloupe:HRO-TYPE-C-31-M-13x -> Connector_Coaxial:U.FL_Hirose_U.FL-R-SMT-1_Vertical
- Q1: value BSS138BKS -> DMP2006UFG; footprint Cantaloupe:SOT-363_SC-70-6 -> Cantaloupe:Diodes_PowerDI3333-8
- R1: footprint Resistor_SMD:R_0402_1005Metric -> Cantaloupe:R_0402_1005Metric
- R2, R6: value 1k -> 10k; footprint Resistor_SMD:R_0402_1005Metric -> Cantaloupe:R_0402_1005Metric
- R3, R5: value 27 -> 10k; footprint Resistor_SMD:R_0402_1005Metric -> Cantaloupe:R_0402_1005Metric
- R4: value 10k -> 470k; footprint Resistor_SMD:R_0402_1005Metric -> Cantaloupe:R_0402_1005Metric
- R7: value 1M -> 10k; footprint Resistor_SMD:R_0402_1005Metric -> Cantaloupe:R_0402_1005Metric
- SW1, SW10, SW11, SW12, SW13, SW14, SW15, SW16, SW17, SW18, SW19, SW2, SW20, SW21, SW22, SW23, SW24, SW25, SW26, SW27, SW28, SW29, SW3, SW30, SW4, SW5, SW6, SW7, SW8, SW9: footprint Cantaloupe:MXOnly-1U-Hotswap-Flippable -> Cantaloupe:MX-Choc-KS27-1U-Hotswap-Flippable
- SW31: value CPG151101S11 -> EVQPUJ; footprint Cantaloupe:MXOnly-1U-Hotswap-Flippable -> Cantaloupe:Panasonic_EVQPUL_EVQPUC; moved to F.Cu
- U1: value ZD25WQ32CEIGR -> MDBT50Q-U1MV2; footprint Cantaloupe:USON-8-1EP_3x2mm_P0.5mm_EP1.6x0.2mm -> Cantaloupe:Raytac_MDBT50Q-U1MV2; moved to F.Cu
- U2: value RP2040 -> TPD4E05U06; footprint Cantaloupe:QFN-56-1EP_7x7mm_P0.4mm_EP3.2x3.2mm_ThermalVias -> Cantaloupe:USON-10_2.5x1.0mm_P0.5mm
- U3: value SN74AHCT1G125 -> nPM1300; footprint Package_TO_SOT_SMD:SOT-353_SC-70-5 -> Cantaloupe:QFN-32-1EP_5x5mm_P0.5mm_EP3.5x3.5mm
- U4: value REF3033 -> TPS61023DRL; footprint Cantaloupe:SOT-23-3 -> Cantaloupe:SOT-563
- U5: value TUSB321 -> SN74AHCT1G125; footprint Cantaloupe:Texas_X2QFN-12_1.6x1.6mm_P0.4mm -> Package_TO_SOT_SMD:SOT-353_SC-70-5
- U6: value 74HC595 -> nRF52840; footprint Cantaloupe:SOIC-16_3.9x9.9mm_P1.27mm -> Cantaloupe:Nordic_AQFN-73-1EP_7x7mm_P0.5mm
- Y1: value 12MHz -> 32M; footprint Crystal:Crystal_SMD_3225-4Pin_3.2x2.5mm -> Crystal:Crystal_SMD_2016-4Pin_2.0x1.6mm
- moved H4 269.3 mm to (200.7, 136.5), turned to 0 degrees
- moved A1 229.4 mm to (133.9, 119.2)
- moved H2 223.6 mm to (193.6, 156.8)
- moved U1 215.0 mm to (15.8, -4.05), turned to 0 degrees
- moved FB1 210.2 mm to (169.8, 48.1)
- moved C15 204.3 mm to (137.3, 132.0)
- moved C14 203.4 mm to (137.3, 129.0)
- moved R6 202.0 mm to (137.3, 130.0), turned to 0 degrees
- moved R5 201.9 mm to (137.3, 128.0)
- moved C23 200.4 mm to (189.2, 58.5), turned to 180 degrees
- moved C30 197.6 mm to (190.4, 65.8), turned to 180 degrees
- moved C31 197.1 mm to (193.5, 66.2), turned to -90 degrees
- moved C22 194.5 mm to (198.6, 57.0)
- moved C29 193.8 mm to (191.1, 57.0), turned to 90 degrees
- moved C28 191.2 mm to (197.8, 57.0)
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- renumbered D31 to D1, D40 to D10, D41 to D11, D42 to D12, D43 to D13, D44 to D14, D45 to D15, D32 to D2, D33 to D3, D34 to D4, D35 to D5, D36 to D6, D37 to D7, D38 to D8, D39 to D9
Connections:
- C10 pad 1: GND -> VBUS_OUT
- C10 pad 2: +3V3 -> GND
- C11 pad 1: GND -> VDD
- C11 pad 2: +3V3 -> GND
- C12 pad 1: GND -> VSYS
- C12 pad 2: +3V3 -> GND
- C13 pad 1: GND -> VSYS
- C13 pad 2: RST -> GND
- C14 pad 2: +3V3 -> Net-(C14-Pad2)
- C15 pad 2: Net-(U2-XIN) -> Net-(C15-Pad2)
- C16 pad 1: GND -> VSYS
- C16 pad 2: +5V -> GND
- C17 pad 1: GND -> +5V
- C17 pad 2: Net-(C17-Pad2) -> GND
- C19 pad 2: +3V3_REF -> Net-(U6-XL1/P0.00)
- C20 pad 2: +3V3_REF -> Net-(U6-XL2/P0.01)
- C21 pad 2: VBUS -> Net-(U6-DECUSB)
- C22 pad 1: GND -> Net-(U6-DEC1)
- C22 pad 2: Net-(D98-K) -> GND
- C23 pad 1: VBUS -> Net-(U6-DEC3)
- C24 pad 1: GND -> /MCU/Ant_2
- C24 pad 2: +5VD -> GND
- C25 pad 1: GND -> /MCU/Ant_Out
- C25 pad 2: +5VD -> GND
- C26 pad 2: +3V3 -> VBUS_OUT
- C27 pad 2: +5VD -> VDD
- C28 pad 1: GND -> VDD
- C28 pad 2: VBUS -> GND
- C29 pad 1: GND -> VDD
- C29 pad 2: /PSU/VBUS_MEAS -> GND
- C3 pad 2: +1V1 -> Net-(U6-XC2)
- C30 pad 1: GND -> VDD
- C30 pad 2: Net-(U9-dVdt) -> GND
- C31 pad 1: +5V -> VDD
- C32 pad 1: +5VD -> Net-(U6-DEC4)
- C33 pad 1: +5VD -> GND
- C33 pad 2: GND -> Net-(U6-DEC4)
- C4 pad 2: +3V3 -> Net-(U6-XC1)
- C5 pad 2: +3V3 -> /IO/~{RST}
- C6 pad 2: +3V3 -> VBUS_RAW
- C7 pad 1: GND -> VBUS
- C7 pad 2: +3V3 -> GND
- C8 pad 1: GND -> VBUS
- C8 pad 2: +3V3 -> GND
- C9 pad 2: +3V3 -> VDD
- D16 pad 1: +5VD -> GND
- D16 pad 2: Net-(D16-DOUT) -> VBUS_RAW
- D17 pad 1: +5VD -> Net-(D17-RK)
- D17 pad 2: Net-(D17-DOUT) -> Net-(D17-GK)
- D17 pad 3: GND -> Net-(D17-BK)
- D17 pad 4: Net-(D16-DOUT) -> VSYS
- FB1 pad 2: Net-(D98-K) -> VBUS_RAW
- H7 pad 1: (no net) -> GND
- J1 pad 1: SWD -> VDD
- J1 pad 2: GND -> SWD
- J1 pad 3: SWC -> /IO/~{RST}
- J2 pad 1: +3V3 -> MOSI
- J2 pad 2: SWD -> SCK
- J2 pad 3: RST -> VDD
- J2 pad 4: SWC -> GND
- J2 pad 5: GND -> NV_~{CS}
- J4 pad 1: +5V -> GND
- J4 pad 2: GND -> CHRG_NTC
- J4 pad 3: /MCU/MOSI -> Net-(J4-Pin_3)
- J4 pad MP: (no net) -> GND
- J5 pad 1: Net-(J5-Pin_1) -> VDD
- J5 pad 2: +5VD -> GND
- J5 pad 3: GND -> VIK_SDA
- J5 pad 4: GND -> VIK_SCL
- Q1 pad 1: GND -> +BATT
- Q1 pad 2: /MCU/1.5A_EN -> +BATT
- Q1 pad 3: Net-(Q1B-D) -> +BATT
- Q1 pad 5: /MCU/3A_EN -> Net-(J4-Pin_3)
- R1 pad 1: +3V3 -> VDD
- R1 pad 2: FLASH_CS -> /IO/CHRG_SCL
- R2 pad 1: FLASH_CS -> VDD
- R2 pad 2: Net-(SW68-B) -> /IO/CHRG_SDA
- R3 pad 1: /MCU/D+ -> VDD
- R3 pad 2: Net-(U2-USB_DP) -> /IO/~{RST}
- R4 pad 1: +3V3 -> GND
- R4 pad 2: RST -> Net-(U3-VSET2)
- R5 pad 1: /MCU/D- -> /MCU/ROTA
- R5 pad 2: Net-(U2-USB_DM) -> Net-(C14-Pad2)
- R6 pad 1: Net-(C17-Pad2) -> Net-(C14-Pad2)
- R6 pad 2: Net-(U2-XOUT) -> VDD
- R7 pad 1: Net-(U5-VBUS_DET) -> VDD
- R7 pad 2: VBUS -> Net-(C15-Pad2)
- SW1 pad 1: COL0 -> /MCU/COL0
- SW10 pad 2: COL1 -> /MCU/COL1
- SW11 pad 1: COL2 -> /MCU/COL2
- SW12 pad 1: COL2 -> /MCU/COL2
- SW13 pad 1: COL2 -> /MCU/COL2
- SW14 pad 1: COL2 -> /MCU/COL2
- SW15 pad 1: COL2 -> /MCU/COL2
- SW16 pad 2: COL3 -> /MCU/COL3
- SW17 pad 2: COL3 -> /MCU/COL3
- SW18 pad 2: COL3 -> /MCU/COL3
- SW19 pad 2: COL3 -> /MCU/COL3
- SW2 pad 1: COL0 -> /MCU/COL0
- SW20 pad 2: COL3 -> /MCU/COL3
- SW21 pad 1: COL4 -> /MCU/COL4
- SW22 pad 1: COL4 -> /MCU/COL4
- SW23 pad 1: COL4 -> /MCU/COL4
- SW24 pad 1: COL4 -> /MCU/COL4
- SW25 pad 1: COL4 -> /MCU/COL4
- SW26 pad 2: COL5 -> /MCU/COL5
- SW27 pad 2: COL5 -> /MCU/COL5
- SW28 pad 2: COL5 -> /MCU/COL5
- SW29 pad 2: COL5 -> /MCU/COL5
- SW3 pad 1: COL0 -> /MCU/COL0
- SW30 pad 2: COL5 -> /MCU/COL5
- SW31 pad 1: Net-(D46A-A) -> GND
- SW31 pad 2: COL6 -> /IO/~{RST}
- SW4 pad 1: COL0 -> /MCU/COL0
- SW5 pad 1: COL0 -> /MCU/COL0
- SW6 pad 2: COL1 -> /MCU/COL1
- SW7 pad 2: COL1 -> /MCU/COL1
- SW8 pad 2: COL1 -> /MCU/COL1
- SW9 pad 2: COL1 -> /MCU/COL1
- U1 pad 1: FLASH_CS -> GND
- U1 pad 2: FLASH_SD1 -> GND
- U1 pad 3: FLASH_SD2 -> /IO/5V_EN
- U1 pad 4: GND -> unconnected-(U1-P1.11(LF)-Pad4)
- U1 pad 5: FLASH_SD0 -> unconnected-(U1-P1.12(LF)-Pad5)
- U1 pad 6: FLASH_CLK -> unconnected-(U1-P1.13(LF)-Pad6)
- U1 pad 7: FLASH_SD3 -> unconnected-(U1-P1.14(LF)-Pad7)
- U1 pad 8: +3V3 -> /MCU/ROW4
- U1 pad 9: GND -> unconnected-(U1-P0.03(LF)/AIN1-Pad9)
- U2 pad 1: +3V3 -> CC1
- U2 pad 10: +3V3 -> CC1
- U2 pad 2: /MCU/TUSB_OUT2 -> /IO/USB_D+
- U2 pad 3: /MCU/TUSB_OUT1 -> GND
- U2 pad 4: unconnected-(U2-GPIO2-Pad4) -> /IO/USB_D-
- U2 pad 5: unconnected-(U2-GPIO3-Pad5) -> CC2
- U2 pad 6: /MCU/ROW0 -> CC2
- U2 pad 7: /MCU/ROW1 -> /IO/USB_D-
- U2 pad 8: /MCU/ROW2 -> GND
- U2 pad 9: /MCU/ROW3 -> /IO/USB_D+
- U3 pad 1: GND -> VSYS
- U3 pad 2: RGB_3V3 -> GND
- U3 pad 3: GND -> unconnected-(U3-SW1-Pad3)
- U3 pad 4: /MCU/RGB_OUT -> VSYS
- U3 pad 5: +5V -> Net-(U3-SW2)
- U4 pad 1: +5V -> Net-(U4-FB)
- U4 pad 2: +3V3_REF -> /IO/5V_EN
- U4 pad 3: GND -> VSYS
- U5 pad 1: CC1 -> GND
- U5 pad 2: CC2 -> Net-(U5-A)
- U5 pad 3: unconnected-(U5-CURRENT_MODE-Pad3) -> GND
- U5 pad 4: GND -> RGB_Out
- U5 pad 5: Net-(U5-VBUS_DET) -> +5V
- Y1 pad 1: Net-(U2-XIN) -> Net-(U6-XC1)
- Y1 pad 3: Net-(C17-Pad2) -> Net-(U6-XC2)
Routing:
- net +5VD: track 668.7 -> 0.00 mm, vias 17 -> 0
- net /MCU/COL0: track 0.00 -> 206.8 mm
- net /MCU/COL1: track 0.00 -> 173.7 mm
- net /MCU/COL2: track 0.00 -> 165.0 mm
- net COL0: track 151.8 -> 0.00 mm
- net /MCU/COL3: track 0.00 -> 151.1 mm
- net /MCU/COL4: track 0.00 -> 147.6 mm
- net /MCU/COL5: track 0.00 -> 112.0 mm
- net COL5: track 104.7 -> 0.00 mm
- net COL4: track 99.6 -> 0.00 mm
- net COL3: track 90.2 -> 0.00 mm
- net /MCU/ROTB: track 0.00 -> 88.7 mm, vias 0 -> 2
- net COL6: track 86.3 -> 0.00 mm
- net /MCU/ROTA: track 0.00 -> 85.8 mm, vias 0 -> 2
- net COL1: track 76.2 -> 0.00 mm
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- added copper zone on B.Cu, net +BATT
- added copper zone on In1.Cu, net GND
- added copper zone on In2.Cu, net GND
- added copper zone on B.Cu, net Net-(J4-Pin_3)
- added copper zone on B.Cu, net Net-(U3-SW2)
- added copper zone on B.Cu, net Net-(U4-FB)
- added copper zone on B.Cu, net Net-(U4-SW)
- added copper zone on F.Cu, net VBUS
- added copper zone on In1.Cu, net VBUS
- added copper zone on B.Cu, net VBUS_OUT
- added copper zone on B.Cu, net VBUS_RAW
- added copper zone on In2.Cu, net VBUS_RAW
- added copper zone on B.Cu, net VDD
- added copper zone on B.Cu, net VSYS
- removed copper zone on F.Cu, net +5V
- removed copper zone on B.Cu, net +5VD
- removed copper zone on F.Cu, net +5VD
- removed copper zone on B.Cu, net /PSU/VBUS_MEAS
- removed copper zone on F.Cu, net GND
- removed copper zone on B.Cu, net Net-(D98-K)
- removed copper zone on F.Cu, net Net-(D98-K)
- removed copper zone on B.Cu, net Net-(U9-ILIM)
Other:
- board size 155.5 x 134.4 mm -> 134 x 122.6 mm
- copper layers 2 -> 4
- board text added: "1"
- board text added: "2"
- board text added: "3"
- board text added: "4"
- board text added: "Cantaloupe V3.0"
- board text added: "J2"
- board text added: "Nice!View"
- board text added: "SW32"
- board text removed: "Honeydew V3.0"
- board text removed: "J4"
