File: PCB/Cantaloupe.kicad_pcb (KiCad board)
At the start: 4 copper layers, 134 x 122.6 mm, 122 parts, among them J1 TC2030-NL, J2 Nice!View, J3 USB_C_Receptacle, J4 Bat, J5 VIK Keyboard, J6 U.FL, Q1 DMP2006UFG, SW1 CPG151101S11, SW10 CPG151101S11, SW11 CPG151101S11, SW12 CPG151101S11, SW13 CPG151101S11, SW14 CPG151101S11, SW15 CPG151101S11, SW16 CPG151101S11, SW17 CPG151101S11, SW18 CPG151101S11, SW19 CPG151101S11, SW2 CPG151101S11, SW20 CPG151101S11, SW21 CPG151101S11, SW22 CPG151101S11, SW23 CPG151101S11, SW24 CPG151101S11, SW25 CPG151101S11, SW26 CPG151101S11, SW27 CPG151101S11, SW28 CPG151101S11, SW29 CPG151101S11, SW3 CPG151101S11, SW30 CPG151101S11, SW31 EVQPUJ, SW32 RotaryEncoder, SW33 Bat_SW, SW4 CPG151101S11, SW5 CPG151101S11, SW6 CPG151101S11, SW7 CPG151101S11, SW8 CPG151101S11, SW9 CPG151101S11, U1 MDBT50Q-U1MV2, U2 TPD4E05U06, U3 nPM1300, U4 TPS61023DRL, U5 SN74AHCT1G125, U6 nRF52840, Y1 32M, Y2 32.768k

Commit message: 24/08/2023 update
Finished routing. Consolidated all libraries into Ariamelon's Kicad Master Library. Added PCM12 switch connected to nPM1300 GPIO. Rearranged components and rerouted.
Parts:
- removed U1: MDBT50Q-U1MV2, Cantaloupe:Raytac_MDBT50Q-U1MV2
- added JP1: 5V_EN, Jumper:SolderJumper-2_P1.3mm_Open_Pad1.0x1.5mm, B.Cu at (203.3, 76.6)
- added R12: 100k, Ariamelon-Device:R_0402_1005Metric, B.Cu at (192.8, 43.6)
- A1: footprint Cantaloupe:Ariamelon_Logo_x2_CU -> Ariamelon-Logo:Ariamelon_Logo_Small_CU
- C10, C14, C15, C18, C19, C20, C21, C22, C23, C24, C25, C26, C27, C28, C29, C3, C30, C31, C32, C33, C4, C5, C6, C8, C9: footprint Cantaloupe:C_0402_1005Metric -> Ariamelon-Device:C_0402_1005Metric
- C11, C12, C13, C16, C7: footprint Cantaloupe:C_0603_1608Metric -> Ariamelon-Device:C_0603_1608Metric
- C17: footprint Cantaloupe:C_0805_2012Metric -> Ariamelon-Device:C_0805_2012Metric
- D1, D10, D11, D12, D13, D14, D15, D2, D3, D4, D5, D6, D7, D8, D9: footprint Cantaloupe:SOT-23-3 -> Ariamelon-Package:SOT-23-3
- D17: footprint Cantaloupe:LED_Lite-On_LTST-S310_3x1.5mm_Horizontal -> Ariamelon-Device:LED_Lite-On_LTST-S310_3x1.5mm_Horizontal
- FB1: footprint Cantaloupe:L_0805_2012Metric -> Ariamelon-Device:L_0805_2012Metric
- H1, H2, H3: footprint Cantaloupe:JLC Tooling Hole -> Ariamelon-HolePad:MountingHole_JLC-Tooling
- H4, H5, H6, H7: footprint Cantaloupe:MountingHole_3.2mm_M3_Pad -> Ariamelon-HolePad:MountingHole_3.2mm_M3_Pad
- J2: footprint Cantaloupe:Nice!View_Flippable -> Ariamelon-Breakout:Breakout_Nice!View_Flippable
- J3: footprint Cantaloupe:HRS_CX70M-24P1 -> Ariamelon-Connector:Hirose_CX70M-24P1
- J4: footprint Cantaloupe:JST_SH_SM03B-SRSS-TB_1x03-1MP_P1.00mm_Horizontal -> Ariamelon-Connector:JST_SH_SM03B-SRSS-TB_1x03-1MP_P1.00mm_Horizontal
- J5: footprint Cantaloupe:VIK-Keyboard-Connector-Horizontal -> Ariamelon-Connector:VIK_Keyboard_Horizontal
- J6: footprint Connector_Coaxial:U.FL_Hirose_U.FL-R-SMT-1_Vertical -> Ariamelon-Connector:U.FL_Hirose_U.FL-R-SMT-1_Vertical
- L1, L2: footprint Cantaloupe:L_Murata_DFE201610P -> Ariamelon-Device:L_Murata_DFE201610P
- L3: footprint Cantaloupe:L_0603_1608Metric -> Ariamelon-Device:L_0603_1608Metric
- L4, L5, L6: footprint Cantaloupe:L_0402_1005Metric -> Ariamelon-Device:L_0402_1005Metric
- Q1: footprint Cantaloupe:Diodes_PowerDI3333-8 -> Ariamelon-Package:Diodes_PowerDI3333-8
- R1, R10, R11, R2, R3, R4, R5, R6, R7, R8, R9: footprint Cantaloupe:R_0402_1005Metric -> Ariamelon-Device:R_0402_1005Metric
- SW1, SW10, SW11, SW12, SW13, SW14, SW15, SW16, SW17, SW18, SW19, SW2, SW20, SW21, SW22, SW23, SW24, SW25, SW26, SW27, SW28, SW29, SW3, SW30, SW4, SW5, SW6, SW7, SW8, SW9: footprint Cantaloupe:MX-Choc-KS27-1U-Hotswap-Flippable -> Ariamelon-Switch:SW_MX-Choc-KS27_1U_Hotswap_Flippable
- SW31: footprint Cantaloupe:Panasonic_EVQPUL_EVQPUC -> Ariamelon-Switch:SW_Panasonic_EVQPUL_EVQPUC
- SW32: footprint Cantaloupe:EVQVVD00203B-Flippable -> Ariamelon-RotaryEncoder:RotaryEncoder_Panasonic_EVQVVD00203B-Flippable
- SW33: value Bat_SW -> SW_SPDT; footprint Button_Switch_SMD:SW_SPDT_PCM12 -> Ariamelon-Switch:SW_CK_SPDT_PCM12
- U2: footprint Cantaloupe:USON-10_2.5x1.0mm_P0.5mm -> Ariamelon-Package:USON-10_2.5x1.0mm_P0.5mm
- U3: footprint Cantaloupe:QFN-32-1EP_5x5mm_P0.5mm_EP3.5x3.5mm -> Ariamelon-Package:QFN-32-1EP_5x5mm_P0.5mm_EP3.5x3.5mm
- U4: footprint Cantaloupe:SOT-563 -> Ariamelon-Package:SOT-563
- U6: footprint Cantaloupe:Nordic_AQFN-73-1EP_7x7mm_P0.5mm -> Ariamelon-Package:Nordic_AQFN-73-1EP_7x7mm_P0.5mm
- Y1: footprint Crystal:Crystal_SMD_2016-4Pin_2.0x1.6mm -> Ariamelon-Device:Crystal_SMD_2016-4Pin_2.0x1.6mm
- Y2: footprint Crystal:Crystal_SMD_2012-2Pin_2.0x1.2mm -> Ariamelon-Device:Crystal_SMD_2012-2Pin_2.0x1.2mm
- moved J6 82.0 mm to (185.9, 57.7), turned to 90 degrees
- moved C25 78.5 mm to (186.3, 59.8), turned to 0 degrees
- moved L6 76.7 mm to (187.2, 60.6), turned to 180 degrees
- moved C24 75.0 mm to (188.4, 60.1), turned to 90 degrees
- moved L5 72.5 mm to (189.6, 60.6), turned to 180 degrees
- moved C10 48.9 mm to (200.0, 67.0), turned to 0 degrees
- moved J1 48.8 mm to (186.1, 65.3), turned to 180 degrees
- moved C5 47.8 mm to (186.4, 69.2), turned to 90 degrees
- moved R3 45.2 mm to (187.2, 69.2), turned to 90 degrees
- moved U5 10.4 mm to (195.9, 73.9), turned to 180 degrees
- moved C18 9.97 mm to (193.9, 73.6), turned to 90 degrees
- moved R1 7.74 mm to (202.0, 53.5), turned to 90 degrees
- moved R2 6.15 mm to (202.0, 51.9), turned to -90 degrees
- moved C26 2.63 mm to (200.0, 66.2)
- moved C4 2.31 mm to (189.6, 55.6)
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Connections:
- C16 pad 1: VSYS -> Net-(JP1-A)
- J1 pad 6: unconnected-(J1-SWO-Pad6) -> /MCU/COL0
- J5 pad 3: VIK_SDA -> /IO/SDA
- J5 pad 4: VIK_SCL -> /IO/SCL
- L2 pad 1: VSYS -> Net-(JP1-A)
- R1 pad 2: /IO/CHRG_SCL -> /IO/SCL
- R2 pad 2: /IO/CHRG_SDA -> /IO/SDA
- R9 pad 1: /IO/5V_EN -> Net-(JP1-A)
- SW33 pad 2: unconnected-(SW33-B-Pad2) -> Net-(SW33-B)
- SW33 pad 3: unconnected-(SW33-C-Pad3) -> nPM_GPIO
- U3 pad 13: /IO/CHRG_SDA -> /IO/SDA
- U3 pad 14: /IO/CHRG_SCL -> /IO/SCL
- U3 pad 8: /IO/CHRG_~{INT} -> nPM_GPIO
- U3 pad 9: unconnected-(U3-GPIO2-Pad9) -> /IO/CHRG_~{INT}
- U4 pad 2: /IO/5V_EN -> Net-(JP1-A)
- U4 pad 3: VSYS -> Net-(JP1-A)
- U6 pad A10: unconnected-(U6-AIN5/P0.29(LF)-PadA10) -> /MCU/ROTA
- U6 pad A12: unconnected-(U6-AIN0/P0.02(LF)-PadA12) -> /MCU/ROTB
- U6 pad A14: unconnected-(U6-P1.15(LF)-PadA14) -> /MCU/ROW3
- U6 pad A16: unconnected-(U6-P1.13(LF)-PadA16) -> /MCU/ROW2
- U6 pad A20: unconnected-(U6-P1.10(LF)-PadA20) -> /MCU/ROW1
- U6 pad A8: unconnected-(U6-AIN7/P0.31(LF)-PadA8) -> /MCU/ROW4
- U6 pad AC21: unconnected-(U6-P0.25-PadAC21) -> /MCU/COL1
- U6 pad AD10: unconnected-(U6-P0.15-PadAD10) -> MOSI
- U6 pad AD16: unconnected-(U6-P0.20-PadAD16) -> VIK_~{CS}
- U6 pad AD18: unconnected-(U6-P0.22-PadAD18) -> MISO
- U6 pad AD20: unconnected-(U6-P0.24-PadAD20) -> SCK
- U6 pad AD22: unconnected-(U6-TRACEDATA0/P1.00/SWO-PadAD22) -> /MCU/COL0
- U6 pad AD8: unconnected-(U6-P0.13-PadAD8) -> NV_~{CS}
- U6 pad G1: /IO/CHRG_SCL -> /IO/CHRG_~{INT}
- U6 pad J24: unconnected-(U6-NFC2/P0.10(LF)-PadJ24) -> /MCU/COL5
- U6 pad L24: unconnected-(U6-NFC1/P0.09(LF)-PadL24) -> /MCU/ROW0
- U6 pad N1: /IO/CHRG_SDA -> /IO/SCL
- U6 pad R1: NV_~{CS} -> /IO/SDA
- U6 pad R24: unconnected-(U6-P1.06(LF)-PadR24) -> /MCU/COL4
- U6 pad U24: unconnected-(U6-P1.04(LF)-PadU24) -> /MCU/COL3
- U6 pad W24: unconnected-(U6-P1.02(LF)-PadW24) -> /MCU/COL2
Routing:
- net VDD: track 65.6 -> 134.8 mm, vias 8 -> 20
- net /IO/SCL: track 0.00 -> 50.3 mm, vias 0 -> 2
- net /IO/~{RST}: track 9.43 -> 59.7 mm, vias 1 -> 5
- net /IO/SDA: track 0.00 -> 49.4 mm, vias 0 -> 2
- net /MCU/ROW3: track 124.8 -> 169.0 mm, vias 0 -> 2
- net /MCU/ROW4: track 145.2 -> 189.3 mm, vias 0 -> 2
- net /MCU/ROTA: track 85.8 -> 129.3 mm, vias 2 -> 4
- net /MCU/ROTB: track 88.7 -> 132.1 mm, vias 2 -> 4
- net VBUS_OUT: track 3.83 -> 40.9 mm, vias 1 -> 4
- net /MCU/ROW2: track 116.3 -> 148.5 mm, vias 0 -> 2
- net GND: track 11.3 -> 39.4 mm, vias 34 -> 109
- net /MCU/ROW1: track 108.5 -> 136.2 mm, vias 0 -> 2
- net VIK_GPIO1: track 2.73 -> 30.1 mm
- net nPM_GPIO: track 0.00 -> 27.3 mm, vias 0 -> 2
- net VIK_GPIO2: track 3.89 -> 30.8 mm
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- added copper zone on F.Cu, net +BATT
- added copper zone on B.Cu, net /MCU/Ant_2
- added copper zone on B.Cu, net /MCU/Ant_Out
- added copper zone on B.Cu, net Net-(JP1-A)
- added copper zone on In1.Cu, net VDD
- added copper zone on In1.Cu, net VSYS
Other:
- outline, holes or cut-outs redrawn
- board text added: "Bat"

Commit message: Cantaloupe V3.0 name changed to CantaloupeBT V1.0 ('BT-V1' branch). Key features updated. Design will be reworked in the coming days!
Parts:
- removed C10, C28, C32, C8: 1u, Ariamelon-Device:C_0402_1005Metric
- removed C11, C12, C13, C16: 10u, Ariamelon-Device:C_0603_1608Metric
- removed C14, C15: 10n, Ariamelon-Device:C_0402_1005Metric
- removed C17: 22u, Ariamelon-Device:C_0805_2012Metric
- removed C18, C22, C29, C30, C31, C33, C5, C9: 100n, Ariamelon-Device:C_0402_1005Metric
- removed C19, C20, C3, C4: 22p, Ariamelon-Device:C_0402_1005Metric
- removed C21, C26, C27: 4u7, Ariamelon-Device:C_0402_1005Metric
- removed C23: 100p, Ariamelon-Device:C_0402_1005Metric
- removed C24: 1p, Ariamelon-Device:C_0402_1005Metric
- removed C25: 1p2, Ariamelon-Device:C_0402_1005Metric
- removed D17: S310F3WT, Ariamelon-Device:LED_Lite-On_LTST-S310_3x1.5mm_Horizontal
- removed J1: TC2030-NL, Connector:Tag-Connect_TC2030-IDC-NL_2x03_P1.27mm_Vertical
- removed J2: Nice!View, Ariamelon-Breakout:Breakout_Nice!View_Flippable
- removed J4: Bat, Ariamelon-Connector:JST_SH_SM03B-SRSS-TB_1x03-1MP_P1.00mm_Horizontal
- removed J6: U.FL, Ariamelon-Connector:U.FL_Hirose_U.FL-R-SMT-1_Vertical
- removed JP1: 5V_EN, Jumper:SolderJumper-2_P1.3mm_Open_Pad1.0x1.5mm
- removed L1: 2u2, Ariamelon-Device:L_Murata_DFE201610P
- removed L2: 470n, Ariamelon-Device:L_Murata_DFE201610P
- removed L3: 10u, Ariamelon-Device:L_0603_1608Metric
- removed L4: 15n, Ariamelon-Device:L_0402_1005Metric
- removed L5: 4n7, Ariamelon-Device:L_0402_1005Metric
- removed L6: 2n2, Ariamelon-Device:L_0402_1005Metric
- removed Q1: DMP2006UFG, Ariamelon-Package:Diodes_PowerDI3333-8
- removed R1, R2, R3, R5, R6, R7, R8: 10k, Ariamelon-Device:R_0402_1005Metric
- removed R10: 732k, Ariamelon-Device:R_0402_1005Metric
- removed R11, R12, R9: 100k, Ariamelon-Device:R_0402_1005Metric
- removed R4: 470k, Ariamelon-Device:R_0402_1005Metric
- removed SW31: EVQPUJ, Ariamelon-Switch:SW_Panasonic_EVQPUL_EVQPUC
- removed SW32: RotaryEncoder, Ariamelon-RotaryEncoder:RotaryEncoder_Panasonic_EVQVVD00203B-Flippable
- removed U3: nPM1300, Ariamelon-Package:QFN-32-1EP_5x5mm_P0.5mm_EP3.5x3.5mm
- removed U4: TPS61023DRL, Ariamelon-Package:SOT-563
- removed U5: SN74AHCT1G125, Package_TO_SOT_SMD:SOT-353_SC-70-5
- removed U6: nRF52840, Ariamelon-Package:Nordic_AQFN-73-1EP_7x7mm_P0.5mm
- removed Y1: 32M, Ariamelon-Device:Crystal_SMD_2016-4Pin_2.0x1.6mm
- removed Y2: 32.768k, Ariamelon-Device:Crystal_SMD_2012-2Pin_2.0x1.2mm
Routing:
- net VDD: track 134.8 -> 0.00 mm, vias 20 -> 0
- net /MCU/ROTB: track 132.1 -> 0.00 mm, vias 4 -> 0
- net /MCU/ROTA: track 129.3 -> 0.00 mm, vias 4 -> 0
- net /IO/~{RST}: track 59.7 -> 0.00 mm, vias 5 -> 0
- net /IO/SCL: track 50.3 -> 0.00 mm, vias 2 -> 0
- net /IO/SDA: track 49.4 -> 0.00 mm, vias 2 -> 0
- net VBUS_OUT: track 40.9 -> 0.00 mm, vias 4 -> 0
- net GND: track 39.4 -> 2.30 mm, vias 109 -> 8
- net /IO/USB_D+: track 51.4 -> 14.7 mm, vias 3 -> 1
- net /IO/USB_D-: track 52.3 -> 15.7 mm, vias 3 -> 1
- net VIK_GPIO2: track 30.8 -> 0.00 mm, vias 2 -> 0
- net VIK_GPIO1: track 30.1 -> 0.00 mm, vias 2 -> 0
- net /MCU/ROW2: track 148.5 -> 119.2 mm, vias 2 -> 0
- net /MCU/ROW3: track 169.0 -> 140.8 mm, vias 2 -> 0
- net /MCU/ROW4: track 189.3 -> 161.9 mm, vias 2 -> 0
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- removed copper zone on B.Cu, net +5V
- removed copper zone on B.Cu, net +BATT
- removed copper zone on F.Cu, net +BATT
- removed copper zone on B.Cu, net /MCU/Ant_2
- removed copper zone on B.Cu, net /MCU/Ant_Out
- removed copper zone on B.Cu, net Net-(J4-Pin_3)
- removed copper zone on B.Cu, net Net-(JP1-A)
- removed copper zone on B.Cu, net Net-(U3-SW2)
- removed copper zone on B.Cu, net Net-(U4-FB)
- removed copper zone on B.Cu, net Net-(U4-SW)
- removed copper zone on F.Cu, net VBUS
- removed copper zone on In1.Cu, net VBUS
- removed copper zone on B.Cu, net VBUS_OUT
- removed copper zone on B.Cu, net VDD
- removed copper zone on In1.Cu, net VDD
- removed copper zone on B.Cu, net VSYS
- removed copper zone on In1.Cu, net VSYS
Other:
- outline, holes or cut-outs redrawn
- board text added: "CantaloupeBT V1.0"
- board text removed: "Bat"
- board text removed: "Cantaloupe V3.0"
- board text removed: "J2"
- board text removed: "Nice!View"
- board text removed: "SW32"
