File: PCB/Cantaloupe.kicad_sch (KiCad schematic)
At the start: 17 parts

Commit message: 23/08/2023 update
Changed MCU to nRF52840. Added nPM1300 PMIC for power management. Replaced SSD1351 display with Nice!View. Added Kailh Choc V1/V2 and Gateron KS-27/KS-33 support.
Parts:
- removed A2: VIK Logo, Cantaloupe:vik-logo-medium, symbol Mechanical:Fiducial
- removed H2 (x4): M3, Cantaloupe:MountingHole_3.2mm_M3_Pad, symbol Mechanical:MountingHole
- removed H2 (x4): M2, MountingHole:MountingHole_2.2mm_M2_Pad, symbol Mechanical:MountingHole
- A1: footprint Cantaloupe:Ariamelon_Logo_x3_Mask -> Ariamelon-Logo:Ariamelon_Logo_Small_CU
- H1, H2: footprint Cantaloupe:MountingHole_3.2mm_M3_Pad -> Ariamelon-HolePad:MountingHole_3.2mm_M3_Pad
- H1, H2, H3: footprint Cantaloupe:JLC Tooling Hole -> Ariamelon-HolePad:MountingHole_JLC-Tooling
- H7: renamed from H11; footprint Cantaloupe:MountingHole_3.2mm_M3_Pad -> Ariamelon-HolePad:MountingHole_3.2mm_M3_Pad; symbol Honeydew:MountingHole_Pad -> Ariamelon-Misc:MountingHole_Pad
Other:
- removed sheet PSU
- removed sheet RGB
- removed sheet USB
- sheet IO ports: added 5V_EN, CHRG_SCL, CHRG_SDA, CHRG_~{INT}, USB_D+, USB_D-, ~{RST}; removed FUSB_1_ID, FUSB_1_OUT1, FUSB_1_OUT2, FUSB_2_ID, FUSB_2_OUT1, FUSB_2_OUT2, IN_D+, IN_D-, OUT_1_D+, OUT_1_D-, OUT_2_D+, OUT_2_D-
- sheet MCU ports: added 5V_EN, CHRG_SCL, CHRG_SDA, CHRG_~{INT}, COL0, COL1, COL2, COL3, COL4, COL5, ROTA, ROTB, USB_D+, USB_D-, ~{RST}; removed 1.5A_EN, 3A_EN, BOARD_ILIM_~{FLT}, BOARD_ISEN, BOARD_VSEN, FUSB_1_ID, FUSB_1_OUT1, FUSB_1_OUT2, FUSB_2_ID, FUSB_2_OUT1, FUSB_2_OUT2, MATRIX_CS, MCU_D+, MCU_D-, MOSI, RGB_IN, RGB_OUT, SCK, ~{RGB_EN}
- sheet Matrix ports: added COL0, COL1, COL2, COL3, COL4, COL5, ROTA, ROTB; removed MATRIX_CS, MOSI, SCK
- moved on the sheet: A1, H1, H2, H3, H7
